File: layouts/default/default.kicad_pcb (KiCad board)
At the start: 2 copper layers, 359 x 111 mm, 181 parts

Commit message: checkin layout
Parts:
- added U14: , CJT_A2541WV_2x5P:HDR-TH_10P-P2.54-V-M-R2-C5-S2.54-1, F.Cu at (260.5, 138.2)
- moved CN3 341.6 mm to (391.8, 143.2), turned to 90 degrees
- moved C11 290.5 mm to (352.1, 77.9)
- moved C12 290.5 mm to (353.0, 88.9)
- moved C13 290.5 mm to (347.7, 86.5)
- moved C14 290.5 mm to (357.5, 83.6)
- moved C15 290.5 mm to (357.4, 79.8)
- moved C16 290.5 mm to (348.8, 78.4)
- moved C17 290.5 mm to (380.3, 79.7)
- moved C18 290.5 mm to (383.1, 77.4)
- moved C19 290.5 mm to (394.5, 85.7)
- moved C20 290.5 mm to (389.0, 88.1)
- moved C21 290.5 mm to (384.7, 86.7)
- moved C22 290.5 mm to (394.4, 80.0)
- moved C23 290.5 mm to (386.8, 77.6)
- moved C24 290.5 mm to (383.9, 81.9)
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Connections:
- net _10 renamed footprint-_10
- R10 pad 1: switches[1]-ethernets[0]-ETH_LED_LINK -> switches[0]-ethernets[2]-ETH_LED_LINK
- R13 pad 1: switches[0]-ethernets[2]-ETH_LED_LINK -> switches[1]-ethernets[0]-ETH_LED_LINK
- R14 pad 1: switches[1]-ethernets[2]-ETH_LED_LINK -> switches[0]-ethernets[3]-ETH_LED_LINK
- R15 pad 1: switches[0]-ethernets[3]-ETH_LED_LINK -> switches[1]-ethernets[2]-ETH_LED_LINK
- R2 pad 1: switches[1]-ethernets[0]-ETH_LED_SPEED -> switches[0]-ethernets[2]-ETH_LED_SPEED
- R5 pad 1: switches[0]-ethernets[2]-ETH_LED_SPEED -> switches[1]-ethernets[0]-ETH_LED_SPEED
- R6 pad 1: switches[1]-ethernets[2]-ETH_LED_SPEED -> switches[0]-ethernets[3]-ETH_LED_SPEED
- R7 pad 1: switches[0]-ethernets[3]-ETH_LED_SPEED -> switches[1]-ethernets[2]-ETH_LED_SPEED
- U2 pad 13: switches[1]-ethernets[0]-ETH_P0_P -> switches[0]-ethernets[2]-ETH_P0_P
- U2 pad 14: switches[1]-ethernets[0]-ETH_P0_N -> switches[0]-ethernets[2]-ETH_P0_N
- U2 pad 15: switches[1]-ethernets[0]-ETH_P1_P -> switches[0]-ethernets[2]-ETH_P1_P
- U2 pad 16: switches[1]-ethernets[0]-ETH_P2_P -> switches[0]-ethernets[2]-ETH_P2_P
- U2 pad 17: switches[1]-ethernets[0]-ETH_P2_N -> switches[0]-ethernets[2]-ETH_P2_N
- U2 pad 18: switches[1]-ethernets[0]-ETH_P1_N -> switches[0]-ethernets[2]-ETH_P1_N
- U2 pad 19: switches[1]-ethernets[0]-ETH_P3_P -> switches[0]-ethernets[2]-ETH_P3_P
- U2 pad 20: switches[1]-ethernets[0]-ETH_P3_N -> switches[0]-ethernets[2]-ETH_P3_N
- U2 pad 49: switches[0]-ethernets[2]-ETH_P0_P -> switches[1]-ethernets[0]-ETH_P0_P
- U2 pad 50: switches[0]-ethernets[2]-ETH_P0_N -> switches[1]-ethernets[0]-ETH_P0_N
- U2 pad 51: switches[0]-ethernets[2]-ETH_P1_P -> switches[1]-ethernets[0]-ETH_P1_P
- U2 pad 52: switches[0]-ethernets[2]-ETH_P2_P -> switches[1]-ethernets[0]-ETH_P2_P
- U2 pad 53: switches[0]-ethernets[2]-ETH_P2_N -> switches[1]-ethernets[0]-ETH_P2_N
- U2 pad 54: switches[0]-ethernets[2]-ETH_P1_N -> switches[1]-ethernets[0]-ETH_P1_N
- U2 pad 55: switches[0]-ethernets[2]-ETH_P3_P -> switches[1]-ethernets[0]-ETH_P3_P
- U2 pad 56: switches[0]-ethernets[2]-ETH_P3_N -> switches[1]-ethernets[0]-ETH_P3_N
- U2 pad 61: switches[1]-ethernets[2]-ETH_P0_P -> switches[0]-ethernets[3]-ETH_P0_P
- U2 pad 62: switches[1]-ethernets[2]-ETH_P0_N -> switches[0]-ethernets[3]-ETH_P0_N
- U2 pad 63: switches[1]-ethernets[2]-ETH_P1_P -> switches[0]-ethernets[3]-ETH_P1_P
- U2 pad 64: switches[1]-ethernets[2]-ETH_P2_P -> switches[0]-ethernets[3]-ETH_P2_P
- U2 pad 65: switches[1]-ethernets[2]-ETH_P2_N -> switches[0]-ethernets[3]-ETH_P2_N
- U2 pad 66: switches[1]-ethernets[2]-ETH_P1_N -> switches[0]-ethernets[3]-ETH_P1_N
- U2 pad 67: switches[1]-ethernets[2]-ETH_P3_P -> switches[0]-ethernets[3]-ETH_P3_P
- U2 pad 68: switches[1]-ethernets[2]-ETH_P3_N -> switches[0]-ethernets[3]-ETH_P3_N
- U2 pad 73: switches[0]-ethernets[3]-ETH_P0_P -> switches[1]-ethernets[2]-ETH_P0_P
- U2 pad 74: switches[0]-ethernets[3]-ETH_P0_N -> switches[1]-ethernets[2]-ETH_P0_N
- U2 pad 75: switches[0]-ethernets[3]-ETH_P1_P -> switches[1]-ethernets[2]-ETH_P1_P
- U2 pad 76: switches[0]-ethernets[3]-ETH_P2_P -> switches[1]-ethernets[2]-ETH_P2_P
- U2 pad 77: switches[0]-ethernets[3]-ETH_P2_N -> switches[1]-ethernets[2]-ETH_P2_N
- U2 pad 78: switches[0]-ethernets[3]-ETH_P1_N -> switches[1]-ethernets[2]-ETH_P1_N
- U2 pad 79: switches[0]-ethernets[3]-ETH_P3_P -> switches[1]-ethernets[2]-ETH_P3_P
- U2 pad 80: switches[0]-ethernets[3]-ETH_P3_N -> switches[1]-ethernets[2]-ETH_P3_N
Other:
- outline, holes or cut-outs redrawn

Commit message: checkin
Parts:
- removed C73, C74: 1µF ±10% 25V X5R, Samsung_Electro_Mechanics_CL05A105KA5NQNC:C0402
- removed R52, R53: 10kΩ ±1% 62.5mW, UNI_ROYAL_0402WGF1002TCE:R0402
- removed U12: , Texas_Instruments_TLV75901PDRVR:WSON-6_L2.0-W2.0-P0.65-TL-EP
- moved R40 231.1 mm to (397.0, 185.8)
- moved R41 231.1 mm to (387.0, 185.8)
- moved R42 231.1 mm to (377.0, 185.8)
- moved R43 231.1 mm to (367.0, 185.8)
- moved R44 231.1 mm to (357.0, 185.8)
- moved R45 231.1 mm to (347.0, 185.8)
- moved R46 231.1 mm to (372.2, 203.2)
- moved R47 231.1 mm to (372.2, 193.2)
- moved R48 231.1 mm to (382.2, 203.2)
- moved R49 231.1 mm to (382.2, 193.2)
- moved R50 231.1 mm to (392.2, 203.2)
- moved R51 231.1 mm to (392.2, 193.2)
- moved R57 231.1 mm to (345.8, 192.8)
- moved R58 231.1 mm to (355.8, 192.8)
- moved R59 231.1 mm to (365.8, 192.8)
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Routing:
- net power_3v3-GND: track 145.2 -> 137.2 mm, vias 66 -> 64
- net power_5v-VCC: track 15.2 -> 11.3 mm
- net power_out-VCC: track 2.74 -> 0.00 mm
- net feedback_divider-output-VDIV_OUTPUT-0: track 2.65 -> 0.00 mm

Commit message: layout checkin
Parts:
- added C100: 100nF ±10% 16V X7R, Samsung_Electro_Mechanics_CL05B104KO5NNNC:C0402, F.Cu at (292.5, 147.0)
- added C73: 18pF ±5% 50V C0G, YAGEO_CC0402JRNPO9BN180:C0402, F.Cu at (393.7, 92.7)
- added C74: 100nF ±10% 16V X7R, Samsung_Electro_Mechanics_CL05B104KO5NNNC:C0402, F.Cu at (382.3, 84.4)
- added C79: 100nF ±10% 16V X7R, Samsung_Electro_Mechanics_CL05B104KO5NNNC:C0402, F.Cu at (392.9, 88.2)
- added C80: 100nF ±10% 16V X7R, Samsung_Electro_Mechanics_CL05B104KO5NNNC:C0402, F.Cu at (387.6, 93.0)
- added C81: 100nF ±10% 16V X7R, Samsung_Electro_Mechanics_CL05B104KO5NNNC:C0402, F.Cu at (386.8, 82.0)
- added C82: 100nF ±10% 16V X7R, Samsung_Electro_Mechanics_CL05B104KO5NNNC:C0402, F.Cu at (392.1, 84.4)
- added C83: 100nF ±10% 16V X7R, Samsung_Electro_Mechanics_CL05B104KO5NNNC:C0402, F.Cu at (382.3, 87.3)
- added C84: 100nF ±10% 16V X7R, Samsung_Electro_Mechanics_CL05B104KO5NNNC:C0402, F.Cu at (382.4, 91.1)
- added C85: 100nF ±10% 16V X7R, Samsung_Electro_Mechanics_CL05B104KO5NNNC:C0402, F.Cu at (391.0, 92.5)
- added C86: 18pF ±5% 50V C0G, YAGEO_CC0402JRNPO9BN180:C0402, F.Cu at (377.9, 90.4)
- added C87: 18pF ±5% 50V C0G, YAGEO_CC0402JRNPO9BN180:C0402, F.Cu at (375.1, 92.7)
- added C88: 100nF ±10% 16V X7R, Samsung_Electro_Mechanics_CL05B104KO5NNNC:C0402, F.Cu at (363.7, 84.4)
- added C89: 100nF ±10% 16V X7R, Samsung_Electro_Mechanics_CL05B104KO5NNNC:C0402, F.Cu at (369.2, 82.0)
- added C90: 100nF ±10% 16V X7R, Samsung_Electro_Mechanics_CL05B104KO5NNNC:C0402, F.Cu at (373.5, 83.4)
- added C91: 100nF ±10% 16V X7R, Samsung_Electro_Mechanics_CL05B104KO5NNNC:C0402, F.Cu at (363.8, 90.1)
- added C92: 100nF ±10% 16V X7R, Samsung_Electro_Mechanics_CL05B104KO5NNNC:C0402, F.Cu at (371.4, 92.5)
- added C93: 100nF ±10% 16V X7R, Samsung_Electro_Mechanics_CL05B104KO5NNNC:C0402, F.Cu at (374.3, 88.2)
- added C94: 100nF ±10% 16V X7R, Samsung_Electro_Mechanics_CL05B104KO5NNNC:C0402, F.Cu at (369.0, 93.0)
- added C95: 100nF ±10% 16V X7R, Samsung_Electro_Mechanics_CL05B104KO5NNNC:C0402, F.Cu at (368.2, 82.0)
- added C96: 100nF ±10% 16V X7R, Samsung_Electro_Mechanics_CL05B104KO5NNNC:C0402, F.Cu at (373.5, 84.4)
- added C97: 100nF ±10% 16V X7R, Samsung_Electro_Mechanics_CL05B104KO5NNNC:C0402, F.Cu at (363.7, 87.3)
- added C98: 100nF ±10% 16V X7R, Samsung_Electro_Mechanics_CL05B104KO5NNNC:C0402, F.Cu at (363.8, 91.1)
- added C99: 100nF ±10% 16V X7R, Samsung_Electro_Mechanics_CL05B104KO5NNNC:C0402, F.Cu at (372.4, 92.5)
- added L1: 10nH ±5% 300mA 300mΩ, FH_VHF201209H10NJT:L0805, F.Cu at (186.2, 110.8)
- added R52: 100kΩ ±1% 62.5mW, UNI_ROYAL_0402WGF1003TCE:R0402, F.Cu at (349.4, 92.8)
- added R53: 10kΩ ±1% 62.5mW, UNI_ROYAL_0402WGF1002TCE:R0402, F.Cu at (351.4, 92.8)
- added R60: 2.49kΩ ±1% 62.5mW, RALEC_RTT022491FTH:R0402, F.Cu at (374.3, 87.2)
- added R61: 10kΩ ±1% 62.5mW, UNI_ROYAL_0402WGF1002TCE:R0402, F.Cu at (367.1, 92.8)
- added R62: 100kΩ ±1% 62.5mW, UNI_ROYAL_0402WGF1003TCE:R0402, F.Cu at (368.1, 92.8)
- added R63: 10kΩ ±1% 62.5mW, UNI_ROYAL_0402WGF1002TCE:R0402, F.Cu at (370.0, 92.8)
- added R64: 10kΩ ±1% 62.5mW, UNI_ROYAL_0402WGF1002TCE:R0402, F.Cu at (366.1, 92.8)
- added R65: 5.1kΩ ±1% 62.5mW, UNI_ROYAL_0402WGF5101TCE:R0402, F.Cu at (288.0, 147.8)
- added R66: 5.1kΩ ±1% 62.5mW, UNI_ROYAL_0402WGF5101TCE:R0402, F.Cu at (293.8, 147.8)
- added U12: , Texas_Instruments_TPS7A4700RGWT:VQFN-20_L5.0-W5.0-P0.65-TL-EP, F.Cu at (247.3, 121.3)
- added U15: , YLPTEC_B0524S_2WR3:PWRM-TH_IBXX05S-2WR3, F.Cu at (252.1, 138.0)
- added U16: , MW_IRM_30_5:PWRM-TH_L69.5-W39.0_LD30-23B05R2, F.Cu at (366.8, 127.8)
- added U17: , Realtek_Semicon_RTL8305NB_VB_CG:QFN-48_L6.0-W6.0-P0.40-TL-EP4.4, F.Cu at (350.2, 87.5)
- added U18: , Realtek_Semicon_RTL8305NB_VB_CG:QFN-48_L6.0-W6.0-P0.40-TL-EP4.4, F.Cu at (387.5, 87.5)
- added U19: , Realtek_Semicon_RTL8305NB_VB_CG:QFN-48_L6.0-W6.0-P0.40-TL-EP4.4, F.Cu at (368.9, 87.5)
- C1: value 22µF ±20% 25V X5R -> 100nF ±10% 16V X7R; footprint Samsung_Electro_Mechanics_CL21A226MAQNNNE:C0805 -> Samsung_Electro_Mechanics_CL05B104KO5NNNC:C0402
- C10: value 100nF ±10% 16V X7R -> 5.6nF ±10% 50V X7R; footprint Samsung_Electro_Mechanics_CL05B104KO5NNNC:C0402 -> YAGEO_CC0402KRX7R9BB562:C0402
- C11: value 100nF ±10% 16V X7R -> 390pF ±10% 50V X7R; footprint Samsung_Electro_Mechanics_CL05B104KO5NNNC:C0402 -> Samsung_Electro_Mechanics_CL05B391KB5NNNC:C0402
- C13: value 100nF ±10% 16V X7R -> 47µF ±20% 35V; footprint Samsung_Electro_Mechanics_CL05B104KO5NNNC:C0402 -> KNSCHA_RVE47UF35V67RV0167:CAP-SMD_BD6.3-L6.6-W6.6-LS7.6-FD
- C14, C15, C16, C39, C42: value 100nF ±10% 16V X7R -> 10µF ±10% 25V X5R; footprint Samsung_Electro_Mechanics_CL05B104KO5NNNC:C0402 -> Samsung_Electro_Mechanics_CL21A106KAYNNNE:C0805
- C17, C3, C32, C4: value 18pF ±5% 50V C0G -> 10µF ±10% 25V X5R; footprint YAGEO_CC0402JRNPO9BN180:C0402 -> Samsung_Electro_Mechanics_CL21A106KAYNNNE:C0805
- C18: value 18pF ±5% 50V C0G -> 100nF ±10% 16V X7R; footprint YAGEO_CC0402JRNPO9BN180:C0402 -> Samsung_Electro_Mechanics_CL05B104KO5NNNC:C0402
- C2: value 22µF ±20% 25V X5R -> 47µF ±20% 35V; footprint Samsung_Electro_Mechanics_CL21A226MAQNNNE:C0805 -> KNSCHA_RVE47UF35V67RV0167:CAP-SMD_BD6.3-L6.6-W6.6-LS7.6-FD
- C28, C29: value 100nF ±10% 16V X7R -> 15pF ±5% 50V C0G; footprint Samsung_Electro_Mechanics_CL05B104KO5NNNC:C0402 -> FH_0402CG150J500NT:C0402
- C30: value 100nF ±10% 16V X7R -> 5.6nF ±10% 50V X7R; footprint Samsung_Electro_Mechanics_CL05B104KO5NNNC:C0402 -> YAGEO_CC0603KRX7R9BB562:C0603
- C31: value 18pF ±5% 50V C0G -> 150pF ±5% 50V C0G; footprint YAGEO_CC0402JRNPO9BN180:C0402 -> YAGEO_CC0603JRNPO9BN151:C0603
- C33, C34, C40, C41, C43, C44: value 100nF ±10% 16V X7R -> 22µF ±20% 6.3V X5R; footprint Samsung_Electro_Mechanics_CL05B104KO5NNNC:C0402 -> Samsung_Electro_Mechanics_CL21A226MQQNNNE:C0805
- C35, C36: value 100nF ±10% 16V X7R -> 10µF ±10% 25V X7R; footprint Samsung_Electro_Mechanics_CL05B104KO5NNNC:C0402 -> Murata_Electronics_GRM21BZ71E106KE15L:C0805
- C37, C38: value 100nF ±10% 16V X7R -> 22µF ±20% 10V X7R; footprint Samsung_Electro_Mechanics_CL05B104KO5NNNC:C0402 -> Murata_Electronics_GRM21BZ71A226ME15L:C0805
- C45, C46: value 22µF ±20% 25V X5R -> 10µF ±10% 25V X5R; footprint Samsung_Electro_Mechanics_CL21A226MAQNNNE:C0805 -> Samsung_Electro_Mechanics_CL21A106KAYNNNE:C0805
- C51, C52, C53: value 100nF ±10% 16V X7R -> 22µF ±20% 25V X5R; footprint Samsung_Electro_Mechanics_CL05B104KO5NNNC:C0402 -> Samsung_Electro_Mechanics_CL21A226MAQNNNE:C0805
- C54: value 10µF ±10% 25V X5R -> 22µF ±20% 25V X5R; footprint Samsung_Electro_Mechanics_CL21A106KAYNNNE:C0805 -> Samsung_Electro_Mechanics_CL21A226MAQNNNE:C0805
- C55, C57: value 10µF ±10% 25V X5R -> 100nF ±10% 16V X7R; footprint Samsung_Electro_Mechanics_CL21A106KAYNNNE:C0805 -> Samsung_Electro_Mechanics_CL05B104KO5NNNC:C0402
- C58: value 10µF ±10% 25V X5R -> 18pF ±5% 50V C0G; footprint Samsung_Electro_Mechanics_CL21A106KAYNNNE:C0805 -> YAGEO_CC0402JRNPO9BN180:C0402
- C59: value 100nF ±10% 16V X7R -> 18pF ±5% 50V C0G; footprint Samsung_Electro_Mechanics_CL05B104KO5NNNC:C0402 -> YAGEO_CC0402JRNPO9BN180:C0402
- C69, C70: value 15pF ±5% 50V C0G -> 100nF ±10% 16V X7R; footprint FH_0402CG150J500NT:C0402 -> Samsung_Electro_Mechanics_CL05B104KO5NNNC:C0402
- C71: value 5.6nF ±10% 50V X7R -> 100nF ±10% 16V X7R; footprint YAGEO_CC0603KRX7R9BB562:C0603 -> Samsung_Electro_Mechanics_CL05B104KO5NNNC:C0402
- C72: value 150pF ±5% 50V C0G -> 18pF ±5% 50V C0G; footprint YAGEO_CC0603JRNPO9BN151:C0603 -> YAGEO_CC0402JRNPO9BN180:C0402
- C75, C76: value 10µF ±10% 25V X7R -> 100nF ±10% 16V X7R; footprint Murata_Electronics_GRM21BZ71E106KE15L:C0805 -> Samsung_Electro_Mechanics_CL05B104KO5NNNC:C0402
- C77, C78: value 22µF ±20% 10V X7R -> 100nF ±10% 16V X7R; footprint Murata_Electronics_GRM21BZ71A226ME15L:C0805 -> Samsung_Electro_Mechanics_CL05B104KO5NNNC:C0402
- R1: value 470Ω ±1% 62.5mW -> 560Ω ±1% 62.5mW; footprint UNI_ROYAL_0402WGF4700TCE:R0402 -> YAGEO_RC0402FR_07560RL:R0402
- R10, R5, R6, R7, R8, R9: value 470Ω ±1% 62.5mW -> 0Ω 62.5mW; footprint UNI_ROYAL_0402WGF4700TCE:R0402 -> UNI_ROYAL_0402WGF0000TCE:R0402
- R11: value 470Ω ±1% 62.5mW -> 100Ω ±1% 62.5mW; footprint UNI_ROYAL_0402WGF4700TCE:R0402 -> UNI_ROYAL_0402WGF1000TCE:R0402
- R12: value 470Ω ±1% 62.5mW -> 0Ω 100mW; footprint UNI_ROYAL_0402WGF4700TCE:R0402 -> UNI_ROYAL_0603WAF0000T5E:R0603
- R13: value 470Ω ±1% 62.5mW -> 4.3kΩ ±1% 100mW; footprint UNI_ROYAL_0402WGF4700TCE:R0402 -> UNI_ROYAL_0603WAF4301T5E:R0603
- R14: value 470Ω ±1% 62.5mW -> 1kΩ ±1% 62.5mW; footprint UNI_ROYAL_0402WGF4700TCE:R0402 -> UNI_ROYAL_0402WGF1001TCE:R0402
- R15, R16: value 470Ω ±1% 62.5mW -> 10kΩ ±1% 62.5mW; footprint UNI_ROYAL_0402WGF4700TCE:R0402 -> UNI_ROYAL_0402WGF1002TCE:R0402
- R17, R18: value 2kΩ ±1% 62.5mW -> 10kΩ ±1% 62.5mW; footprint UNI_ROYAL_0402WGF2001TCE:R0402 -> UNI_ROYAL_0402WGF1002TCE:R0402
- R19: value 2.49kΩ ±1% 62.5mW -> 10kΩ ±1% 62.5mW; footprint RALEC_RTT022491FTH:R0402 -> UNI_ROYAL_0402WGF1002TCE:R0402
- R2: value 470Ω ±1% 62.5mW -> 100kΩ ±1% 62.5mW; footprint UNI_ROYAL_0402WGF4700TCE:R0402 -> UNI_ROYAL_0402WGF1003TCE:R0402
- R21, R26: value 100kΩ ±1% 62.5mW -> 0Ω 62.5mW; footprint UNI_ROYAL_0402WGF1003TCE:R0402 -> UNI_ROYAL_0402WGF0000TCE:R0402
- R22, R23, R25: value 10kΩ ±1% 62.5mW -> 0Ω 62.5mW; footprint UNI_ROYAL_0402WGF1002TCE:R0402 -> UNI_ROYAL_0402WGF0000TCE:R0402
- R24: value 2.49kΩ ±1% 62.5mW -> 0Ω 62.5mW; footprint RALEC_RTT022491FTH:R0402 -> UNI_ROYAL_0402WGF0000TCE:R0402
- R27: value 10kΩ ±1% 62.5mW -> 10Ω ±1% 62.5mW; footprint UNI_ROYAL_0402WGF1002TCE:R0402 -> UNI_ROYAL_0402WGF100JTCE:R0402
- R28, R30, R32, R33, R40, R41, R42, R43: value 10kΩ ±1% 62.5mW -> 470Ω ±1% 62.5mW; footprint UNI_ROYAL_0402WGF1002TCE:R0402 -> UNI_ROYAL_0402WGF4700TCE:R0402
- R29: value 2.49kΩ ±1% 62.5mW -> 470Ω ±1% 62.5mW; footprint RALEC_RTT022491FTH:R0402 -> UNI_ROYAL_0402WGF4700TCE:R0402
- R3, R4: value 470Ω ±1% 62.5mW -> 2kΩ ±1% 62.5mW; footprint UNI_ROYAL_0402WGF4700TCE:R0402 -> UNI_ROYAL_0402WGF2001TCE:R0402
- R31: value 100kΩ ±1% 62.5mW -> 470Ω ±1% 62.5mW; footprint UNI_ROYAL_0402WGF1003TCE:R0402 -> UNI_ROYAL_0402WGF4700TCE:R0402
- R34: value 100Ω ±1% 62.5mW -> 470Ω ±1% 62.5mW; footprint UNI_ROYAL_0402WGF1000TCE:R0402 -> UNI_ROYAL_0402WGF4700TCE:R0402
- R35: value 0Ω 100mW -> 470Ω ±1% 62.5mW; footprint UNI_ROYAL_0603WAF0000T5E:R0603 -> UNI_ROYAL_0402WGF4700TCE:R0402
- R36, R37: value 5.1kΩ ±1% 62.5mW -> 470Ω ±1% 62.5mW; footprint UNI_ROYAL_0402WGF5101TCE:R0402 -> UNI_ROYAL_0402WGF4700TCE:R0402
- R38: value 4.3kΩ ±1% 100mW -> 470Ω ±1% 62.5mW; footprint UNI_ROYAL_0603WAF4301T5E:R0603 -> UNI_ROYAL_0402WGF4700TCE:R0402
- R39: value 1kΩ ±1% 62.5mW -> 470Ω ±1% 62.5mW; footprint UNI_ROYAL_0402WGF1001TCE:R0402 -> UNI_ROYAL_0402WGF4700TCE:R0402
- R46: value 0Ω 62.5mW -> 47kΩ ±1% 62.5mW; footprint UNI_ROYAL_0402WGF0000TCE:R0402 -> UNI_ROYAL_0402WGF4702TCE:R0402
- R50: value 0Ω 62.5mW -> 2.49kΩ ±1% 62.5mW; footprint UNI_ROYAL_0402WGF0000TCE:R0402 -> RALEC_RTT022491FTH:R0402
- R51, R58, R59: value 0Ω 62.5mW -> 10kΩ ±1% 62.5mW; footprint UNI_ROYAL_0402WGF0000TCE:R0402 -> UNI_ROYAL_0402WGF1002TCE:R0402
- R55: value 10kΩ ±1% 62.5mW -> 2.49kΩ ±1% 62.5mW; footprint UNI_ROYAL_0402WGF1002TCE:R0402 -> RALEC_RTT022491FTH:R0402
- R56: value 47kΩ ±1% 62.5mW -> 10kΩ ±1% 62.5mW; footprint UNI_ROYAL_0402WGF4702TCE:R0402 -> UNI_ROYAL_0402WGF1002TCE:R0402
- R57: value 0Ω 62.5mW -> 100kΩ ±1% 62.5mW; footprint UNI_ROYAL_0402WGF0000TCE:R0402 -> UNI_ROYAL_0402WGF1003TCE:R0402
- REF**: renamed from PS3; value (none) -> CONN-TH_NC3MAAH
- REF**: renamed from PS6; value (none) -> CONN-TH_NC3MAAH
- REF**: renamed from PS9; value (none) -> CONN-TH_NC3MAAH
- REF**: renamed from PS2; value (none) -> CONN-TH_NCJ6FA-H
- REF**: renamed from PS7; value (none) -> CONN-TH_NC3MAAH
- REF**: renamed from PS4; value (none) -> CONN-TH_NC3MAAH
- REF**: renamed from PS1; value (none) -> CONN-TH_NCJ6FA-H
- REF**: renamed from PS5; value (none) -> CONN-TH_NC3MAAH
- REF**: renamed from PS8; value (none) -> CONN-TH_NC3MAAH
- REF**: renamed from PS12; value (none) -> CONN-TH_NCJ6FA-H
- REF**: renamed from PS10; value (none) -> CONN-TH_NC3MAAH
- REF**: renamed from PS11; value (none) -> CONN-TH_NC3MAAH
- U1: footprint Texas_Instruments_SN74LVC1G07DBVR:SOT-23-5_L3.0-W1.7-P0.95-LS2.8-BR -> Analog_Devices_AD1938WBSTZ_RL:LQFP-48_L7.0-W7.0-P0.50-LS9.0-BL
- U10: footprint Realtek_Semicon_RTL8305NB_VB_CG:QFN-48_L6.0-W6.0-P0.40-TL-EP4.4 -> Texas_Instruments_TPS7A4700RGWT:VQFN-20_L5.0-W5.0-P0.65-TL-EP
- U11: footprint Analog_Devices_ADAU1452WBCPZ:LFCSP-72_L10.0-W10.0-P0.50-LS10.2-BL-EP5.3 -> TEXAS_INSTRUMENTS_TPSM863257RDXR:QFN-7_L4.0-W3.3_TPSM863257RDXR
- U13: footprint TEXAS_INSTRUMENTS_TPSM863257RDXR:QFN-7_L4.0-W3.3_TPSM863257RDXR -> Texas_Instruments_TPS7A4700RGWT:VQFN-20_L5.0-W5.0-P0.65-TL-EP
- U14: footprint CJT_A2541WV_2x5P:HDR-TH_10P-P2.54-V-M-R2-C5-S2.54-1 -> YLPTEC_B0524S_2WR3:PWRM-TH_IBXX05S-2WR3
- U2: footprint HCTL_HC_RJ45_059C_2_4_1:RJ45-TH_HC-RJ45-059C-2X4-1 -> Texas_Instruments_SN74LVC1G07DBVR:SOT-23-5_L3.0-W1.7-P0.95-LS2.8-BR
- U7: footprint MW_IRM_30_5:PWRM-TH_L69.5-W39.0_LD30-23B05R2 -> Analog_Devices_ADAU1452WBCPZ:LFCSP-72_L10.0-W10.0-P0.50-LS10.2-BL-EP5.3
- U8: footprint Realtek_Semicon_RTL8305NB_VB_CG:QFN-48_L6.0-W6.0-P0.40-TL-EP4.4 -> CJT_A2541WV_2x5P:HDR-TH_10P-P2.54-V-M-R2-C5-S2.54-1
- U9: footprint Realtek_Semicon_RTL8305NB_VB_CG:QFN-48_L6.0-W6.0-P0.40-TL-EP4.4 -> HCTL_HC_RJ45_059C_2_4_1:RJ45-TH_HC-RJ45-059C-2X4-1
- X1: footprint Yangxing_Tech_X322525MRB4SI:OSC-SMD_4P-L3.2-W2.5-BL_SIT8008BI -> TAE_TXM12_288M0004322FBCDO00T:CRYSTAL-SMD_4P-L3.2-W2.5-BL-2
- X4: footprint TAE_TXM12_288M0004322FBCDO00T:CRYSTAL-SMD_4P-L3.2-W2.5-BL-2 -> Yangxing_Tech_X322525MRB4SI:OSC-SMD_4P-L3.2-W2.5-BL_SIT8008BI
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Connections:
- net SCLK renamed spi0-SCLK
- net cm5-pins[26] renamed pins[26]
- net hdmi1-pins[48] renamed pins[48]
- net switches[2]-ethernets[0]-ETH_LED_SPEED renamed switches[2]-ethernets[4]-ETH_LED_SPEED
- net switches[2]-ethernets[0]-ETH_P2_N renamed switches[2]-ethernets[4]-ETH_P2_N
- net switches[2]-ethernets[0]-ETH_P2_P renamed switches[2]-ethernets[4]-ETH_P2_P
- net switches[2]-ethernets[0]-ETH_P3_N renamed switches[2]-ethernets[4]-ETH_P3_N
- net switches[2]-ethernets[0]-ETH_P3_P renamed switches[2]-ethernets[4]-ETH_P3_P
- net switches[2]-ethernets[3]-ETH_P0_P renamed footprint-NR-2
- C1 pad 1: power_5v-VCC -> CM
- C10 pad 1: switches[0]-_power_1v2-VCC -> ad1938-net
- C11 pad 1: power_3v3-VCC -> LF
- C12 pad 1: power_3v3-VCC -> FILTR
- C13 pad 1: power_3v3-VCC -> FILTR
- C16 pad 1: power_3v3-VCC -> power_digital-VCC
- C17 pad 1: crystal-XI-1 -> power_3v3-VCC
- C18 pad 1: crystal-XO-1 -> power_3v3-VCC
- C19 pad 1: switches[1]-_power_1v2-VCC -> power_digital-VCC
- C2 pad 1: power_5v-VCC -> CM
- C20 pad 1: switches[1]-_power_1v2-VCC -> power_digital-VCC
- C21 pad 1: switches[1]-_power_1v2-VCC -> power_digital-VCC
- C22 pad 1: switches[1]-_power_1v2-VCC -> power_digital-VCC
- C23 pad 1: switches[1]-_power_1v2-VCC -> power_3v3-VCC
- C24 pad 1: switches[1]-_power_1v2-VCC -> power_3v3-VCC
- C28 pad 1: power_3v3-VCC -> nOE
- C29 pad 1: power_3v3-VCC -> XTALOUT
- C3 pad 1: crystal-XI-0 -> power_analog-VCC
- C30 pad 1: power_3v3-VCC -> c1-net
- C30 pad 2: power_3v3-GND -> power_3v3-VCC
- C31 pad 1: crystal-XI-2 -> PLLFILT
- C31 pad 2: power_3v3-GND -> power_3v3-VCC
- C32 pad 1: crystal-XO-2 -> power_5v-VCC
- C33 pad 1: switches[2]-_power_1v2-VCC -> regulator_3v3_analog-power_out-VCC
- C34 pad 1: switches[2]-_power_1v2-VCC -> regulator_3v3_analog-power_out-VCC
- C35 pad 1: switches[2]-_power_1v2-VCC -> power_5v-VCC
- C36 pad 1: switches[2]-_power_1v2-VCC -> power_5v-VCC
- C37 pad 1: switches[2]-_power_1v2-VCC -> power_3v3-VCC
- C38 pad 1: switches[2]-_power_1v2-VCC -> power_3v3-VCC
- C39 pad 1: power_3v3-VCC -> regulator_24v_isolated_neg-power_out-VCC
- C39 pad 2: power_3v3-GND -> regulator_24v_isolated_neg-power_out-GND
- C4 pad 1: crystal-XO-0 -> regulator_3v3_analog-power_out-VCC
- C40 pad 1: power_3v3-VCC -> regulator_24v_isolated_pos-power_out-GND
- C40 pad 2: power_3v3-GND -> regulator_24v_isolated_neg-power_out-GND
- C41 pad 1: power_3v3-VCC -> regulator_24v_isolated_pos-power_out-GND
- C41 pad 2: power_3v3-GND -> regulator_24v_isolated_neg-power_out-GND
- C42 pad 1: power_3v3-VCC -> regulator_24v_isolated_pos-power_out-VCC
- C42 pad 2: power_3v3-GND -> regulator_24v_isolated_pos-power_out-GND
- C43 pad 1: power_3v3-VCC -> regulator_18v_pos-power_out-VCC
- C43 pad 2: power_3v3-GND -> regulator_24v_isolated_pos-power_out-GND
- C44 pad 1: power_3v3-VCC -> regulator_18v_pos-power_out-VCC
- C44 pad 2: power_3v3-GND -> regulator_24v_isolated_pos-power_out-GND
- C45 pad 1: power_5v-VCC -> regulator_24v_isolated_neg-power_out-VCC
- C45 pad 2: power_3v3-GND -> regulator_24v_isolated_neg-power_out-GND
- C46 pad 1: power_5v-VCC -> regulator_24v_isolated_pos-power_out-VCC
- C46 pad 2: power_3v3-GND -> regulator_24v_isolated_pos-power_out-GND
- C5 pad 1: switches[0]-_power_1v2-VCC -> power_analog-VCC
- C54 pad 1: power_3v3-VCC -> power_5v-VCC
- C55 pad 1: power_3v3-VCC -> power_5v-VCC
- C57 pad 1: power_digital-VCC -> power_5v-VCC
- C58 pad 1: power_3v3-VCC -> crystal-XI-0
- C59 pad 1: power_3v3-VCC -> crystal-XO-0
- C6 pad 1: switches[0]-_power_1v2-VCC -> power_analog-VCC
- C60 pad 1: power_digital-VCC -> switches[0]-_power_1v2-VCC
- C61 pad 1: power_digital-VCC -> switches[0]-_power_1v2-VCC
- C62 pad 1: power_digital-VCC -> switches[0]-_power_1v2-VCC
- C63 pad 1: power_digital-VCC -> switches[0]-_power_1v2-VCC
- C64 pad 1: power_3v3-VCC -> switches[0]-_power_1v2-VCC
- C65 pad 1: power_3v3-VCC -> switches[0]-_power_1v2-VCC
- C69 pad 1: nOE -> power_3v3-VCC
- C7 pad 1: switches[0]-_power_1v2-VCC -> power_analog-VCC
- C70 pad 1: XTALOUT -> power_3v3-VCC
- C71 pad 1: c1-net -> power_3v3-VCC
- C71 pad 2: power_3v3-VCC -> power_3v3-GND
- C72 pad 1: PLLFILT -> crystal-XI-1
- C72 pad 2: power_3v3-VCC -> power_3v3-GND
- C75 pad 1: power_5v-VCC -> switches[1]-_power_1v2-VCC
- C76 pad 1: power_5v-VCC -> switches[1]-_power_1v2-VCC
- C77 pad 1: power_3v3-VCC -> switches[1]-_power_1v2-VCC
- C78 pad 1: power_3v3-VCC -> switches[1]-_power_1v2-VCC
- C8 pad 1: switches[0]-_power_1v2-VCC -> power_analog-VCC
- C9 pad 1: switches[0]-_power_1v2-VCC -> regulator_3v3_analog-power_out-VCC
- CN1 pad 13: pins[25] -> cm5_i2s_resistor_jumpers[4]-logic_out-line
- CN1 pad 2: switches[2]-ethernets[0]-ETH_P1_P -> switches[2]-ethernets[4]-ETH_P1_P
- CN1 pad 3: switches[2]-ethernets[0]-ETH_P1_N -> switches[2]-ethernets[4]-ETH_P1_N
- CN1 pad 5: switches[2]-ethernets[0]-ETH_P0_N -> switches[2]-ethernets[4]-ETH_P0_N
- CN1 pad 6: switches[2]-ethernets[0]-ETH_P0_P -> switches[2]-ethernets[4]-ETH_P0_P
- CN1 pad 76: gpio[18]-pins[48] -> cm5_i2s_resistor_jumpers[3]-logic_out-line
- CN1 pad 87: led_data-pins[26] -> cm5_i2s_resistor_jumpers[5]-logic_out-line
- CN1 pad 93: switches[2]-ethernets[0]-ETH_LED_LINK -> switches[2]-ethernets[4]-ETH_LED_LINK
- R1 pad 1: switches[0]-ethernets[0]-ETH_LED_SPEED -> LF
- R1 pad 2: _12 -> ad1938-net
- R10 pad 1: switches[0]-ethernets[2]-ETH_LED_LINK -> model-i2s_outs[0]-SD-1
- R10 pad 2: _22 -> cm5_i2s_resistor_jumpers[5]-logic_out-line
- R11 pad 1: switches[0]-ethernets[1]-ETH_LED_LINK -> XTALIN_MCLK
- R11 pad 2: _34 -> nOE
- R12 pad 1: switches[1]-ethernets[1]-ETH_LED_LINK -> collector
- R12 pad 2: _46 -> power_digital-VCC
- R13 pad 1: switches[1]-ethernets[0]-ETH_LED_LINK -> PLLFILT
- R13 pad 2: _59 -> c1-net
- R14 pad 1: switches[0]-ethernets[3]-ETH_LED_LINK -> power_3v3-VCC
- R14 pad 2: _71 -> VDRIVE
- R15 pad 1: switches[1]-ethernets[2]-ETH_LED_LINK -> logic_out-SCL
- R15 pad 2: _83 -> power_3v3-VCC
- R16 pad 1: switches[1]-ethernets[3]-ETH_LED_LINK -> reset_resistor_jumpers[0]-logic_out-SDA
- R16 pad 2: _95 -> power_3v3-VCC
- R17 pad 1: activity_led-cathode -> i2c_resistor_jumpers[1]-i2c_out-SCL
- R17 pad 2: activity_led_resistor-pins[20] -> power_3v3-VCC
- R18 pad 1: cm5-cathode -> reset_resistor_jumpers[2]-logic_out-SDA
- R18 pad 2: Y -> power_3v3-VCC
- R19 pad 1: footprint-IBREF-0 -> i2c_resistor_jumpers[2]-i2c_out-SCL
- R19 pad 2: power_3v3-GND -> power_3v3-VCC
- R2 pad 1: switches[0]-ethernets[2]-ETH_LED_SPEED -> nPD_nRST
- R2 pad 2: _24 -> power_3v3-GND
- R20 pad 1: switches[0]-loop_indication-LDIND_DIS_LD -> i2c_out-SDA
- R21 pad 1: switches[0]-ethernets[0]-ETH_LED_LINK -> switches[0]-i2c_mdio-SCL
- R21 pad 2: power_3v3-GND -> logic_out-SCL
- R22 pad 1: switches[0]-ethernets[2]-ETH_LED_LINK -> switches[0]-i2c_mdio-SDA
- R22 pad 2: power_3v3-VCC -> reset_resistor_jumpers[0]-logic_out-SDA
- R23 pad 1: switches[0]-reset-RESETB -> switches[1]-i2c_mdio-SCL
- R23 pad 2: power_3v3-VCC -> i2c_resistor_jumpers[1]-i2c_out-SCL
- R24 pad 1: footprint-IBREF-1 -> switches[1]-i2c_mdio-SDA
- R24 pad 2: power_3v3-GND -> reset_resistor_jumpers[2]-logic_out-SDA
- R25 pad 1: switches[1]-loop_indication-LDIND_DIS_LD -> switches[2]-i2c_mdio-SCL
- R25 pad 2: power_3v3-VCC -> i2c_resistor_jumpers[2]-i2c_out-SCL
- R26 pad 1: switches[1]-ethernets[0]-ETH_LED_LINK -> switches[2]-i2c_mdio-SDA
- R26 pad 2: power_3v3-GND -> i2c_out-SDA
- R27 pad 1: switches[1]-ethernets[2]-ETH_LED_LINK -> power_3v3-GND
- R27 pad 2: power_3v3-VCC -> regulator_24v_isolated_pos-power_out-GND
- R28 pad 1: switches[1]-reset-RESETB -> switches[0]-ethernets[3]-ETH_LED_SPEED
- R28 pad 2: power_3v3-VCC -> _12
- R29 pad 1: footprint-IBREF-2 -> switches[0]-ethernets[1]-ETH_LED_SPEED
- R29 pad 2: power_3v3-GND -> _24
- R3 pad 1: switches[0]-ethernets[1]-ETH_LED_SPEED -> activity_led-cathode
- R3 pad 2: _36 -> activity_led_resistor-pins[20]
- R30 pad 1: switches[2]-loop_indication-LDIND_DIS_LD -> switches[1]-ethernets[3]-ETH_LED_SPEED
- R30 pad 2: power_3v3-VCC -> _36
- R31 pad 1: switches[2]-ethernets[0]-ETH_LED_LINK -> switches[1]-ethernets[1]-ETH_LED_SPEED
- R31 pad 2: power_3v3-GND -> _48
- R32 pad 1: switches[2]-ethernets[2]-ETH_LED_LINK -> switches[0]-ethernets[4]-ETH_LED_SPEED
- R32 pad 2: power_3v3-VCC -> _57
- R33 pad 1: switches[2]-reset-RESETB -> switches[0]-ethernets[2]-ETH_LED_SPEED
- R33 pad 2: power_3v3-VCC -> _69
- R34 pad 1: XTALIN_MCLK -> switches[1]-ethernets[2]-ETH_LED_SPEED
- R34 pad 2: nOE -> _81
- R35 pad 1: collector -> ethernets[0]-ETH_LED_SPEED
- R35 pad 2: power_digital-VCC -> _93
- R36 pad 1: cc[0]-line -> switches[0]-ethernets[3]-ETH_LED_LINK
- R36 pad 2: power_3v3-GND -> footprint-_10
- R37 pad 1: cc[1]-line -> switches[0]-ethernets[1]-ETH_LED_LINK
- R37 pad 2: power_3v3-GND -> _22
- R38 pad 1: PLLFILT -> switches[1]-ethernets[3]-ETH_LED_LINK
- R38 pad 2: c1-net -> _34
- R39 pad 1: power_3v3-VCC -> switches[1]-ethernets[1]-ETH_LED_LINK
- R39 pad 2: VDRIVE -> _46
- R4 pad 1: switches[1]-ethernets[1]-ETH_LED_SPEED -> cm5-cathode
- R4 pad 2: _48 -> Y
- R40 pad 1: logic_out-SCL -> switches[0]-ethernets[4]-ETH_LED_LINK
- R40 pad 2: power_3v3-VCC -> _59
- R41 pad 1: reset_resistor_jumpers[0]-logic_out-SDA -> switches[0]-ethernets[2]-ETH_LED_LINK
- R41 pad 2: power_3v3-VCC -> _71
- R42 pad 1: i2c_resistor_jumpers[1]-i2c_out-SCL -> switches[1]-ethernets[2]-ETH_LED_LINK
- R42 pad 2: power_3v3-VCC -> _83
- R43 pad 1: reset_resistor_jumpers[2]-logic_out-SDA -> switches[1]-ethernets[0]-ETH_LED_LINK
- R43 pad 2: power_3v3-VCC -> _95
- R44 pad 1: i2c_resistor_jumpers[2]-i2c_out-SCL -> power_5v-VCC
- R44 pad 2: power_3v3-VCC -> EN
- R45 pad 1: i2c_out-SDA -> VDIV_OUTPUT
- R45 pad 2: power_3v3-VCC -> power_3v3-GND
- R46 pad 1: switches[0]-i2c_mdio-SCL -> power_3v3-VCC
- R46 pad 2: logic_out-SCL -> VDIV_OUTPUT
- R47 pad 1: switches[0]-i2c_mdio-SDA -> switches[0]-reset-RESETB
- R48 pad 1: switches[1]-i2c_mdio-SCL -> switches[1]-reset-RESETB
- R48 pad 2: i2c_resistor_jumpers[1]-i2c_out-SCL -> logic_out-SCL
- R49 pad 1: switches[1]-i2c_mdio-SDA -> switches[2]-reset-RESETB
- R5 pad 1: switches[1]-ethernets[0]-ETH_LED_SPEED -> model-i2s_ins[0]-SCK-1
- R5 pad 2: _57 -> cm5_i2s_resistor_jumpers[3]-logic_out-line
- R50 pad 1: switches[2]-i2c_mdio-SCL -> footprint-IBREF-0
- R50 pad 2: i2c_resistor_jumpers[2]-i2c_out-SCL -> power_3v3-GND
- R51 pad 1: switches[2]-i2c_mdio-SDA -> switches[0]-loop_indication-LDIND_DIS_LD
- R51 pad 2: i2c_out-SDA -> power_3v3-VCC
- R54 pad 1: power_5v-VCC -> switches[0]-reset-RESETB
- R54 pad 2: EN -> power_3v3-VCC
- R55 pad 1: feedback_divider-output-VDIV_OUTPUT-1 -> footprint-IBREF-1
- R56 pad 1: power_3v3-VCC -> switches[1]-loop_indication-LDIND_DIS_LD
- R56 pad 2: feedback_divider-output-VDIV_OUTPUT-1 -> power_3v3-VCC
- R57 pad 1: switches[0]-reset-RESETB -> switches[1]-ethernets[0]-ETH_LED_LINK
- R57 pad 2: reset_resistor_jumpers[0]-logic_out-SDA -> power_3v3-GND
- R58 pad 1: switches[1]-reset-RESETB -> switches[1]-ethernets[2]-ETH_LED_LINK
- R58 pad 2: logic_out-SCL -> power_3v3-VCC
- R59 pad 1: switches[2]-reset-RESETB -> switches[1]-reset-RESETB
- R59 pad 2: reset_resistor_jumpers[2]-logic_out-SDA -> power_3v3-VCC
- R6 pad 1: switches[0]-ethernets[3]-ETH_LED_SPEED -> model-i2s_ins[0]-WS-1
- R6 pad 2: _69 -> cm5_i2s_resistor_jumpers[4]-logic_out-line
- R7 pad 1: switches[1]-ethernets[2]-ETH_LED_SPEED -> model-i2s_ins[0]-SD-1
- R7 pad 2: _81 -> pins[24]
- R8 pad 1: switches[1]-ethernets[3]-ETH_LED_SPEED -> model-i2s_outs[0]-SCK-1
- R8 pad 2: _93 -> cm5_i2s_resistor_jumpers[3]-logic_out-line
- R9 pad 1: switches[0]-ethernets[0]-ETH_LED_LINK -> model-i2s_outs[0]-WS-1
- R9 pad 2: footprint-_10 -> cm5_i2s_resistor_jumpers[4]-logic_out-line
- REF** pad : footprint-net-3 -> (no net)
- REF** pad : footprint-net-6 -> (no net)
- REF** pad : footprint-net-9 -> (no net)
- REF** pad : footprint-net-7 -> (no net)
- REF** pad : footprint-net-4 -> (no net)
- REF** pad : footprint-net-5 -> (no net)
- REF** pad : footprint-net-8 -> (no net)
- REF** pad : footprint-net-10 -> (no net)
- REF** pad : footprint-net-11 -> (no net)
- U1 pad 1: N_C_ -> power_3v3-GND
- U1 pad 2: input-pins[94] -> MCLKI_XI
- U1 pad 3: power_3v3-GND -> MCLKO_XO
- U1 pad 4: Y -> power_3v3-GND
- U1 pad 5: power_3v3-VCC -> power_analog-VCC
- U10 pad 1: switches[2]-_power_1v2-VCC -> regulator_3v3_analog-power_out-VCC
- U10 pad 10: switches[2]-ethernets[2]-ETH_P1_N -> P0P4V
- U10 pad 11: switches[2]-ethernets[2]-ETH_P0_N -> power_3v3-GND
- U10 pad 12: switches[2]-ethernets[2]-ETH_P0_P -> power_3v3-GND
- U10 pad 13: switches[2]-_power_1v2-VCC -> power_5v-VCC
- U10 pad 15: switches[2]-ethernets[3]-ETH_P0_N -> power_5v-VCC
- U10 pad 16: switches[2]-ethernets[3]-ETH_P1_N -> power_5v-VCC
- U10 pad 17: switches[2]-ethernets[3]-ETH_P1_P -> footprint-net-11
- U10 pad 18: power_3v3-VCC -> footprint-net-12
- U10 pad 19: switches[2]-ethernets[4]-ETH_P1_P -> footprint-net-9
- U10 pad 2: switches[2]-ethernets[2]-ETH_P0_P -> footprint-net-10
- U10 pad 20: switches[2]-ethernets[4]-ETH_P1_N -> regulator_3v3_analog-power_out-VCC
- U10 pad 21: switches[2]-ethernets[4]-ETH_P0_N -> footprint-EP-2
- U10 pad 3: switches[2]-ethernets[2]-ETH_P0_N -> footprint-SENSE_FB-2
- U10 pad 4: switches[2]-ethernets[2]-ETH_P1_N -> P6P4V2
- U10 pad 5: switches[2]-ethernets[2]-ETH_P1_P -> P6P4V1
- U10 pad 6: power_3v3-VCC -> P3P2V
- U10 pad 7: switches[2]-_power_1v2-VCC -> power_3v3-GND
- U10 pad 8: power_3v3-VCC -> power_3v3-GND
- U10 pad 9: switches[2]-ethernets[2]-ETH_P1_P -> P0P8V
- U11 pad 1: power_3v3-GND -> power_5v-VCC
- U11 pad 2: power_3v3-VCC -> SW
- U11 pad 3: VDRIVE -> power_3v3-VCC
- U11 pad 4: SPDIFIN -> power_3v3-GND
- U11 pad 5: SPDIFOUT -> PG
- U11 pad 6: power_3v3-GND -> EN
- U11 pad 7: power_3v3-VCC -> VDIV_OUTPUT
- U13 pad 1: power_5v-VCC -> regulator_18v_pos-power_out-VCC
- U13 pad 2: SW -> footprint-net-6
- U13 pad 3: power_3v3-VCC -> footprint-SENSE_FB-1
- U13 pad 4: power_3v3-GND -> regulator_24v_isolated_pos-power_out-GND
- U13 pad 5: PG -> regulator_24v_isolated_pos-power_out-GND
- U13 pad 6: EN -> regulator_24v_isolated_pos-power_out-GND
- U13 pad 7: feedback_divider-output-VDIV_OUTPUT-1 -> regulator_24v_isolated_pos-power_out-GND
- U14 pad 1: _1 -> power_5v-VCC
- U14 pad 2: logic_out-SCL -> power_3v3-GND
- U14 pad 4: reset_resistor_jumpers[0]-logic_out-SDA -> regulator_24v_isolated_neg-power_out-GND
- U14 pad 6: _6 -> regulator_24v_isolated_neg-power_out-VCC
- U2 pad 1: switches[0]-ethernets[0]-ETH_P0_P -> N_C_
- U2 pad 2: switches[0]-ethernets[0]-ETH_P0_N -> input-pins[94]
- U2 pad 3: switches[0]-ethernets[0]-ETH_P1_P -> power_3v3-GND
- U2 pad 4: switches[0]-ethernets[0]-ETH_P2_P -> Y
- U2 pad 5: switches[0]-ethernets[0]-ETH_P2_N -> power_3v3-VCC
- U7 pad 1: AL_L -> power_3v3-GND
- U7 pad 2: neutral -> power_3v3-VCC
- U7 pad 3: power_5v-VCC -> VDRIVE
- U7 pad 4: power_3v3-GND -> SPDIFIN
- U8 pad 1: switches[0]-_power_1v2-VCC -> _1
- U8 pad 10: switches[0]-ethernets[2]-ETH_P1_N -> dsp_debug_connector-_10
- U8 pad 2: switches[0]-ethernets[1]-ETH_P0_P -> logic_out-SCL
- U8 pad 3: switches[0]-ethernets[1]-ETH_P0_N -> _3
- U8 pad 4: switches[0]-ethernets[1]-ETH_P1_N -> reset_resistor_jumpers[0]-logic_out-SDA
- U8 pad 5: switches[0]-ethernets[1]-ETH_P1_P -> reset_resistor_jumpers[0]-logic_out-SDA
- U8 pad 6: power_3v3-VCC -> _6
- U8 pad 7: switches[0]-_power_1v2-VCC -> _7
- U8 pad 8: power_3v3-VCC -> _8
- U8 pad 9: switches[0]-ethernets[2]-ETH_P1_P -> power_3v3-GND
- U9 pad 1: switches[1]-_power_1v2-VCC -> switches[0]-ethernets[3]-ETH_P0_P
- U9 pad 10: switches[1]-ethernets[2]-ETH_P1_N -> footprint-_10
- U9 pad 11: switches[1]-ethernets[2]-ETH_P0_N -> power_3v3-GND
- U9 pad 12: switches[1]-ethernets[2]-ETH_P0_P -> _12
- U9 pad 13: switches[1]-_power_1v2-VCC -> switches[0]-ethernets[1]-ETH_P0_P
- U9 pad 14: switches[1]-ethernets[3]-ETH_P0_P -> switches[0]-ethernets[1]-ETH_P0_N
- U9 pad 15: switches[1]-ethernets[3]-ETH_P0_N -> switches[0]-ethernets[1]-ETH_P1_P
- U9 pad 16: switches[1]-ethernets[3]-ETH_P1_N -> switches[0]-ethernets[1]-ETH_P2_P
- U9 pad 17: switches[1]-ethernets[3]-ETH_P1_P -> switches[0]-ethernets[1]-ETH_P2_N
- U9 pad 18: power_3v3-VCC -> switches[0]-ethernets[1]-ETH_P1_N
- U9 pad 19: switches[1]-ethernets[4]-ETH_P1_P -> switches[0]-ethernets[1]-ETH_P3_P
- U9 pad 2: switches[1]-ethernets[1]-ETH_P0_P -> switches[0]-ethernets[3]-ETH_P0_N
- U9 pad 20: switches[1]-ethernets[4]-ETH_P1_N -> switches[0]-ethernets[1]-ETH_P3_N
- U9 pad 21: switches[1]-ethernets[4]-ETH_P0_N -> power_3v3-GND
- U9 pad 22: switches[1]-ethernets[4]-ETH_P0_P -> _22
- U9 pad 23: switches[1]-_power_1v2-VCC -> power_3v3-GND
- U9 pad 24: switches[1]-_power_1v2-VCC -> _24
- U9 pad 25: switches[1]-i2c_mdio-SCL -> switches[1]-ethernets[3]-ETH_P0_P
- U9 pad 26: switches[1]-i2c_mdio-SDA -> switches[1]-ethernets[3]-ETH_P0_N
- U9 pad 27: switches[1]-reset-RESETB -> switches[1]-ethernets[3]-ETH_P1_P
- U9 pad 28: switches[1]-loop_indication-LDIND_DIS_LD -> switches[1]-ethernets[3]-ETH_P2_P
- U9 pad 29: switches[1]-ethernets[0]-ETH_LED_LINK -> switches[1]-ethernets[3]-ETH_P2_N
- U9 pad 3: switches[1]-ethernets[1]-ETH_P0_N -> switches[0]-ethernets[3]-ETH_P1_P
- U9 pad 30: switches[1]-ethernets[1]-ETH_LED_LINK -> switches[1]-ethernets[3]-ETH_P1_N
- U9 pad 31: power_3v3-VCC -> switches[1]-ethernets[3]-ETH_P3_P
- U9 pad 32: switches[1]-ethernets[2]-ETH_LED_LINK -> switches[1]-ethernets[3]-ETH_P3_N
- U9 pad 33: switches[1]-ethernets[3]-ETH_LED_LINK -> power_3v3-GND
- U9 pad 34: switches[1]-ethernets[4]-ETH_LED_LINK -> _34
- U9 pad 35: switches[1]-_power_1v2-VCC -> power_3v3-GND
- U9 pad 36: switches[1]-_power_1v2-VCC -> _36
- U9 pad 37: power_3v3-VCC -> switches[1]-ethernets[1]-ETH_P0_P
- U9 pad 38: power_3v3-VCC -> switches[1]-ethernets[1]-ETH_P0_N
- U9 pad 39: crystal-XO-1 -> switches[1]-ethernets[1]-ETH_P1_P
- U9 pad 4: switches[1]-ethernets[1]-ETH_P1_N -> switches[0]-ethernets[3]-ETH_P2_P
- U9 pad 40: crystal-XI-1 -> switches[1]-ethernets[1]-ETH_P2_P
- U9 pad 41: switches[1]-_power_1v2-VCC -> switches[1]-ethernets[1]-ETH_P2_N
- U9 pad 42: footprint-IBREF-1 -> switches[1]-ethernets[1]-ETH_P1_N
- U9 pad 43: switches[1]-_power_1v2-VCC -> switches[1]-ethernets[1]-ETH_P3_P
- U9 pad 44: switches[1]-ethernets[0]-ETH_P0_P -> switches[1]-ethernets[1]-ETH_P3_N
- U9 pad 45: switches[1]-ethernets[0]-ETH_P0_N -> power_3v3-GND
- U9 pad 46: switches[1]-ethernets[0]-ETH_P1_N -> _46
- U9 pad 47: switches[1]-ethernets[0]-ETH_P1_P -> power_3v3-GND
- U9 pad 48: power_3v3-VCC -> _48
- U9 pad 49: power_3v3-GND -> switches[0]-ethernets[4]-ETH_P0_P
- U9 pad 5: switches[1]-ethernets[1]-ETH_P1_P -> switches[0]-ethernets[3]-ETH_P2_N
- U9 pad 6: power_3v3-VCC -> switches[0]-ethernets[3]-ETH_P1_N
- U9 pad 7: switches[1]-_power_1v2-VCC -> switches[0]-ethernets[3]-ETH_P3_P
- U9 pad 8: power_3v3-VCC -> switches[0]-ethernets[3]-ETH_P3_N
- U9 pad 9: switches[1]-ethernets[2]-ETH_P1_P -> power_3v3-GND
- X1 pad 1: crystal-XI-0 -> nOE
- X1 pad 3: crystal-XO-0 -> XTALOUT
- X2 pad 1: crystal-XI-1 -> crystal-XI-0
- X2 pad 3: crystal-XO-1 -> crystal-XO-0
- X3 pad 1: crystal-XI-2 -> crystal-XI-1
- X3 pad 3: crystal-XO-2 -> crystal-XO-1
- X4 pad 1: nOE -> crystal-XI-2
- X4 pad 3: XTALOUT -> crystal-XO-2
Routing:
- net (no net): track 102.2 -> 0.00 mm
- net switches[0]-ethernets[4]-ETH_P1_P: track 0.00 -> 41.9 mm, vias 0 -> 1
- net switches[0]-ethernets[4]-ETH_P1_N: track 0.00 -> 41.8 mm, vias 0 -> 1
- net power_3v3-GND: track 137.2 -> 178.7 mm, vias 64 -> 88
- net switches[0]-ethernets[2]-ETH_P0_N: track 0.00 -> 40.8 mm, vias 0 -> 1
- net switches[0]-ethernets[2]-ETH_P0_P: track 0.00 -> 40.8 mm, vias 0 -> 1
- net switches[0]-ethernets[4]-ETH_P0_P: track 0.00 -> 39.6 mm, vias 0 -> 1
- net switches[0]-ethernets[4]-ETH_P0_N: track 0.00 -> 39.5 mm, vias 0 -> 1
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
Commit message: ethernet layout
Parts:
- moved U8 108.2 mm to (164.0, 117.5)
- moved U15 55.1 mm to (253.5, 82.9), turned to 180 degrees
- moved R5 48.6 mm to (159.0, 97.0), turned to 90 degrees
- moved U14 48.5 mm to (253.5, 90.2), turned to 180 degrees
- moved C46 47.0 mm to (241.0, 80.5), turned to 90 degrees
- moved U13 44.4 mm to (236.8, 80.5), turned to -90 degrees
- moved C44 42.5 mm to (232.2, 80.5), turned to -90 degrees
- moved C43 42.0 mm to (230.2, 80.5), turned to -90 degrees
- moved C42 41.6 mm to (228.2, 80.5), turned to -90 degrees
- moved C45 38.3 mm to (241.0, 87.8), turned to 90 degrees
- moved U12 35.2 mm to (236.8, 87.7), turned to -90 degrees
- moved C41 32.8 mm to (232.4, 87.7), turned to -90 degrees
- moved C40 32.1 mm to (230.4, 87.7), turned to -90 degrees
- moved R7 31.9 mm to (158.0, 99.5)
- moved C39 31.5 mm to (228.4, 87.7), turned to -90 degrees
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- renumbered REF** to J1000, REF** to J1001, REF** to J1002, REF** to J1003, REF** to J1004, REF** to J1005, REF** to J1006, REF** to J1007, REF** to J1008, REF** to J1009, REF** to J1010, REF** to J1011
Routing:
- net switches[1]-ethernets[0]-ETH_P0_P: track 0.00 -> 31.6 mm, vias 0 -> 1
- net switches[1]-ethernets[0]-ETH_P1_N: track 0.00 -> 31.4 mm, vias 0 -> 1
- net switches[1]-ethernets[0]-ETH_P1_P: track 0.00 -> 31.3 mm, vias 0 -> 1
- net switches[1]-ethernets[3]-ETH_P0_N: track 0.00 -> 30.7 mm, vias 0 -> 1
- net switches[1]-ethernets[3]-ETH_P0_P: track 0.00 -> 30.7 mm, vias 0 -> 1
- net switches[1]-ethernets[0]-ETH_P0_N: track 0.00 -> 30.4 mm, vias 0 -> 1
- net switches[1]-ethernets[2]-ETH_P1_P: track 0.00 -> 30.2 mm, vias 0 -> 1
- net switches[1]-ethernets[2]-ETH_P1_N: track 0.00 -> 26.4 mm, vias 0 -> 1
- net switches[1]-ethernets[3]-ETH_P1_N: track 0.00 -> 26.4 mm
- net switches[1]-ethernets[3]-ETH_P1_P: track 0.00 -> 26.4 mm
- net switches[1]-ethernets[2]-ETH_P0_N: track 0.00 -> 26.2 mm, vias 0 -> 1
- net switches[1]-ethernets[2]-ETH_P0_P: track 0.00 -> 26.0 mm
- net switches[1]-ethernets[1]-ETH_P0_N: track 0.00 -> 19.9 mm, vias 0 -> 1
- net switches[1]-ethernets[1]-ETH_P0_P: track 0.00 -> 19.8 mm, vias 0 -> 1
- net switches[1]-ethernets[1]-ETH_P1_N: track 0.00 -> 19.2 mm
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Other:
- outline, holes or cut-outs redrawn
