File: projects/unreleased-packages/ti-drv135/layouts/driver/driver.kicad_pcb (KiCad board)
At the start: 2 copper layers, 12 parts

Commit message: wiggly in place
Routing:
- net audio_out_P: track 0.00 -> 10.6 mm, vias 0 -> 1
- net audio_out_N: track 0.00 -> 10.5 mm, vias 0 -> 1
- net anode_P: track 15.1 -> 19.1 mm, vias 0 -> 1
- net anode_N: track 14.7 -> 18.6 mm, vias 0 -> 1
Changed lines of the file:
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@@
+	)
+	(segment
+		(start 168.9 123.7)
+		(end 167 121.8)
+		(width 0.124)
+		(layer "F.Cu")
+		(net 1)
+	)
+	(segment
+		(start 167 121.8)
+		(end 159.1 121.8)
+		(width 0.124)
+		(layer "F.Cu")
+		(net 1)
+	)
+	(via
+		(at 168.9 123.7)
+		(size 1.8)
+		(drill 1)
+		(layers "F.Cu" "B.Cu")
+		(net 1)
+	)
+	(segment
+		(start 167.1 120)
+		(end 159.1 120)
+		(width 0.124)
+		(layer "F.Cu")
+		(net 2)
+	)
+	(segment
+		(start 168.8 118.3)
+		(end 167.1 120)
+		(width 0.124)
+		(layer "F.Cu")
+		(net 2)
+	)
+	(segment
+		(start 168.9 118.3)
+		(end 168.8 118.3)
+		(width 0.124)
+		(layer "F.Cu")
+		(net 2)
+	)
+	(via
+		(at 168.9 118.3)
+		(size 1.8)
+		(drill 1)
+		(layers "F.Cu" "B.Cu")
+		(net 2)
 	)
 	(segment
@@
 	)
 	(segment
+		(start 155.4 118.3)
+		(end 153.9 118.3)
+		(width 0.124)
+		(layer "F.Cu")
+		(net 8)
+	)
+	(segment
 		(start 152.03 118.53)
 		(end 151.9 118.4)
@@
 	)
 	(segment
+		(start 157.1 120)
+		(end 155.4 118.3)
+		(width 0.124)
+		(layer "F.Cu")
+		(net 8)
+	)
+	(segment
 		(start 146.345005 119.492005)
 		(end 146.345005 118.29)
@@
 		(net 8)
 	)
+	(via
+		(at 153.9 118.3)
+		(size 1.8)
+		(drill 1)
+		(layers "F.Cu" "B.Cu")
+		(net 8)
+	)
 	(segment
 		(start 145.065005 117.434995)
@@
 	)
 	(segment
+		(start 155.2 123.7)
+		(end 153.9 123.7)
+		(width 0.124)
+		(layer "F.Cu")
+		(net 11)
+	)
+	(segment
 		(start 152.874 121.256)
 		(end 156.356 121.256)
@@
 		(net 11)
 	)
+	(segment
+		(start 157.1 121.8)
+		(end 155.2 123.7)
+		(width 0.124)
+		(layer "F.Cu")
+		(net 11)
+	)
+	(via
+		(at 153.9 123.7)
+		(size 1.8)
+		(drill 1)
+		(layers "F.Cu" "B.Cu")
+		(net 11)
+	)
