File: projects/dsp/layouts/default/default.kicad_pcb (KiCad board)
At the start: 2 copper layers, 359 x 111 mm, 313 parts

Commit message: wiggly in place
Parts:
- removed D1: , Everlight_Elec_19_213_Y2C_CQ2R2L_3T_CY:LED0603-RD-YELLOW
- removed D2: , Hubei_KENTO_Elec_KT_0603G:LED0603-RD
- removed SW1, SW2: , XKB_Connectivity_TS_1101_C_W:SW-SMD_L6.0-W3.3-LS8.0
- added C157: 4.7µF ±5% 100V, XIAMEN_FARATRONIC_C232A475J6SC000:CAP-TH_L17.5-W8.5-P15.00-D0.8, F.Cu at (52.0, 130.8)
- added C158: 4.7µF ±5% 100V, XIAMEN_FARATRONIC_C232A475J6SC000:CAP-TH_L17.5-W8.5-P15.00-D0.8, F.Cu at (43.3, 130.8)
- added C159: 4.7µF ±5% 100V, XIAMEN_FARATRONIC_C232A475J6SC000:CAP-TH_L17.5-W8.5-P15.00-D0.8, F.Cu at (76.0, 130.8)
- added C160: 4.7µF ±5% 100V, XIAMEN_FARATRONIC_C232A475J6SC000:CAP-TH_L17.5-W8.5-P15.00-D0.8, F.Cu at (67.4, 130.8)
- C28, C29: value 15pF ±5% 50V C0G -> 100nF ±10% 16V X7R; footprint FH_0402CG150J500NT:C0402 -> Samsung_Electro_Mechanics_CL05B104KO5NNNC:C0402
- C47, C48, C49, C50, C51, C52, C53, C54: value 22µF ±20% 25V X5R -> 22µF ±20% 6.3V X5R; footprint Samsung_Electro_Mechanics_CL21A226MAQNNNE:C0805 -> Samsung_Electro_Mechanics_CL21A226MQQNNNE:C0805
- R17, R18, R19, R20: value 10kΩ ±1% 62.5mW -> 1.5kΩ ±1% 62.5mW; footprint UNI_ROYAL_0402WGF1002TCE:R0402 -> UNI_ROYAL_0402WGF1501TCE:R0402
- R21, R22: value 0Ω 62.5mW -> 1.5kΩ ±1% 62.5mW; footprint UNI_ROYAL_0402WGF0000TCE:R0402 -> UNI_ROYAL_0402WGF1501TCE:R0402
- R27: value 10Ω ±1% 62.5mW -> 10kΩ ±1% 62.5mW; footprint UNI_ROYAL_0402WGF100JTCE:R0402 -> UNI_ROYAL_0402WGF1002TCE:R0402
- R3: value 2kΩ ±1% 62.5mW -> 0Ω 62.5mW; footprint UNI_ROYAL_0402WGF2001TCE:R0402 -> UNI_ROYAL_0402WGF0000TCE:R0402
- R4: value 2kΩ ±1% 62.5mW -> 10kΩ ±1% 62.5mW; footprint UNI_ROYAL_0402WGF2001TCE:R0402 -> UNI_ROYAL_0402WGF1002TCE:R0402
- R45: value 10kΩ ±1% 62.5mW -> 0Ω 62.5mW; footprint UNI_ROYAL_0402WGF1002TCE:R0402 -> UNI_ROYAL_0402WGF0000TCE:R0402
- R46: value 47kΩ ±1% 62.5mW -> 0Ω 62.5mW; footprint UNI_ROYAL_0402WGF4702TCE:R0402 -> UNI_ROYAL_0402WGF0000TCE:R0402
- U2: footprint Texas_Instruments_SN74LVC1G07DBVR:SOT-23-5_L3.0-W1.7-P0.95-LS2.8-BR -> cm5:cm5
- moved CN3 436.0 mm to (-16.5, 13.0), turned to 0 degrees
- moved R22 395.5 mm to (0.00, -70.0), turned to 0 degrees
- moved R23 390.1 mm to (24.6, -45.0), turned to 0 degrees
- moved R21 389.5 mm to (0.00, -60.0), turned to 0 degrees
- moved R24 378.9 mm to (22.6, -16.0), turned to 0 degrees
- moved R20 376.4 mm to (0.00, -50.0)
- moved R19 365.3 mm to (0.00, -40.0), turned to 0 degrees
- moved R26 362.0 mm to (20.0, -10.0), turned to 0 degrees
- moved R25 357.3 mm to (20.0, 0.00), turned to 0 degrees
- moved R18 356.2 mm to (0.00, -30.0), turned to 0 degrees
- moved R17 351.4 mm to (0.00, -20.0), turned to 0 degrees
- moved R3 345.8 mm to (16.4, -13.0), turned to 0 degrees
- moved R46 338.2 mm to (30.0, -10.0), turned to 0 degrees
- moved C55 332.8 mm to (90.0, -55.1), turned to 0 degrees
- moved R45 331.2 mm to (30.1, 0.70), turned to 0 degrees
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Connections:
- net cm5-pins[15]-0 renamed fan_tacho-pins[15]
- net cm5-pins[15]-1 renamed cm5-pins[15]
- net cm5-pins[17]-0 renamed ethernet_sync-pins[17]
- net cm5-pins[17]-1 renamed cm5-pins[17]
- net cm5-pins[93]-0 renamed usb_cc[0]-pins[93]
- net cm5-pins[93]-1 renamed cm5-pins[93]
- net cm5-pins[95]-0 renamed usb_cc[1]-pins[95]
- net cm5-pins[95]-1 renamed cm5-pins[95]
- net cm5_i2s_resistor_jumpers[3]-logic_out-line renamed logic_out-SCK
- net cm5_i2s_resistor_jumpers[4]-logic_out-line renamed logic_out-WS
- net cm5_i2s_resistor_jumpers[5]-logic_out-line renamed cm5_i2s_resistor_jumpers[5]-logic_out-SD
- net hdmi0-HDMI_D0_N renamed hdmis[0]-HDMI_D0_N
- net hdmi0-HDMI_D0_P renamed hdmis[0]-HDMI_D0_P
- net hdmi0-HDMI_D1_N renamed hdmis[0]-HDMI_D1_N
- net hdmi0-HDMI_D1_P renamed hdmis[0]-HDMI_D1_P
- net hdmi0-HDMI_D2_N renamed hdmis[0]-HDMI_D2_N
- net hdmi0-HDMI_D2_P renamed hdmis[0]-HDMI_D2_P
- net hdmi0-SCL renamed hdmis[0]-SCL
- net hdmi0-SDA renamed hdmis[0]-SDA
- net hdmi1-HDMI_D0_N renamed hdmis[1]-HDMI_D0_N
- net hdmi1-HDMI_D0_P renamed hdmis[1]-HDMI_D0_P
- net hdmi1-HDMI_D1_N renamed hdmis[1]-HDMI_D1_N
- net hdmi1-HDMI_D1_P renamed hdmis[1]-HDMI_D1_P
- net hdmi1-HDMI_D2_N renamed hdmis[1]-HDMI_D2_N
- net hdmi1-HDMI_D2_P renamed hdmis[1]-HDMI_D2_P
- net hdmi1-SCL renamed hdmis[1]-SCL
- net hdmi1-SDA renamed hdmis[1]-SDA
- net pins[24] renamed cm5_i2s_resistor_jumpers[2]-logic_out-SD
- net regulator_18v_pos-power_out-VCC renamed power_18v_pos
- net regulator_24v_isolated_neg-power_out-GND renamed power_18v_neg
- net regulator_3v3_analog-power_out-VCC renamed power_3v3_analog
- net spi0-MISO renamed spis[0]-MISO
- net spi0-MOSI renamed spis[0]-MOSI
- net spi0-SCLK renamed spis[0]-SCLK
- net spi0_cs0-pins[38] renamed spi0_cs[0]-pins[38]
- net usb3_0-USB_D_N renamed usb3[0]-USB_D_N
- net usb3_0-USB_D_P renamed usb3[0]-USB_D_P
- net usb3_1-USB_D_N renamed usb3[1]-USB_D_N
- net usb3_1-USB_D_P renamed usb3[1]-USB_D_P
- C100 pad 1: power_5v-VCC -> power_5v
- C104 pad 1: regulator_24v_isolated_pos-power_out-GND -> power_out-GND
- C105 pad 2: regulator_24v_isolated_pos-power_out-GND -> power_out-GND
- C111 pad 1: regulator_24v_isolated_pos-power_out-GND -> power_out-GND
- C112 pad 2: regulator_24v_isolated_pos-power_out-GND -> power_out-GND
- C118 pad 1: regulator_24v_isolated_pos-power_out-GND -> power_out-GND
- C119 pad 2: regulator_24v_isolated_pos-power_out-GND -> power_out-GND
- C125 pad 1: regulator_24v_isolated_pos-power_out-GND -> power_out-GND
- C126 pad 2: regulator_24v_isolated_pos-power_out-GND -> power_out-GND
- C132 pad 1: regulator_24v_isolated_pos-power_out-GND -> power_out-GND
- C133 pad 2: regulator_24v_isolated_pos-power_out-GND -> power_out-GND
- C139 pad 1: regulator_24v_isolated_pos-power_out-GND -> power_out-GND
- C14 pad 1: power_3v3-VCC -> power_3v3_digital
- C140 pad 2: regulator_24v_isolated_pos-power_out-GND -> power_out-GND
- C146 pad 1: regulator_24v_isolated_pos-power_out-GND -> power_out-GND
- C147 pad 2: regulator_24v_isolated_pos-power_out-GND -> power_out-GND
- C15 pad 1: power_3v3-VCC -> power_3v3_digital
- C153 pad 1: regulator_24v_isolated_pos-power_out-GND -> power_out-GND
- C154 pad 2: regulator_24v_isolated_pos-power_out-GND -> power_out-GND
- C17 pad 1: power_3v3-VCC -> power_3v3_digital
- C18 pad 1: power_3v3-VCC -> power_3v3_digital
- C23 pad 1: power_3v3-VCC -> power_3v3_digital
- C24 pad 1: power_3v3-VCC -> power_3v3_digital
- C25 pad 1: power_3v3-VCC -> power_3v3_digital
- C26 pad 1: power_3v3-VCC -> power_3v3_digital
- C27 pad 1: power_3v3-VCC -> power_3v3_digital
- C30 pad 2: power_3v3-VCC -> power_3v3_digital
- C31 pad 2: power_3v3-VCC -> power_3v3_digital
- C32 pad 1: power_5v-VCC -> power_5v
- C35 pad 1: power_5v-VCC -> power_5v
- C36 pad 1: power_5v-VCC -> power_5v
- C37 pad 1: power_3v3-VCC -> power_3v3_digital
- C38 pad 1: power_3v3-VCC -> power_3v3_digital
- C40 pad 1: regulator_24v_isolated_pos-power_out-GND -> power_out-GND
- C41 pad 1: regulator_24v_isolated_pos-power_out-GND -> power_out-GND
- C42 pad 2: regulator_24v_isolated_pos-power_out-GND -> power_out-GND
- C43 pad 2: regulator_24v_isolated_pos-power_out-GND -> power_out-GND
- C44 pad 2: regulator_24v_isolated_pos-power_out-GND -> power_out-GND
- C46 pad 2: regulator_24v_isolated_pos-power_out-GND -> power_out-GND
- C47 pad 1: power_5v-VCC -> power_5v
- C48 pad 1: power_5v-VCC -> power_5v
- C49 pad 1: power_5v-VCC -> power_5v
- C50 pad 1: power_5v-VCC -> power_5v
- C51 pad 1: power_5v-VCC -> power_5v
- C52 pad 1: power_5v-VCC -> power_5v
- C53 pad 1: power_5v-VCC -> power_5v
- C54 pad 1: power_5v-VCC -> power_5v
- C55 pad 1: power_5v-VCC -> power_5v
- C56 pad 1: power_5v-VCC -> power_5v
- C57 pad 1: power_5v-VCC -> power_5v
- C66 pad 1: power_3v3-VCC -> power_3v3_digital
- C67 pad 1: power_3v3-VCC -> power_3v3_digital
- C68 pad 1: power_3v3-VCC -> power_3v3_digital
- C69 pad 1: power_3v3-VCC -> power_3v3_digital
- C70 pad 1: power_3v3-VCC -> power_3v3_digital
- C71 pad 1: power_3v3-VCC -> power_3v3_digital
- C80 pad 1: power_3v3-VCC -> power_3v3_digital
- C81 pad 1: power_3v3-VCC -> power_3v3_digital
- C82 pad 1: power_3v3-VCC -> power_3v3_digital
- C83 pad 1: power_3v3-VCC -> power_3v3_digital
- C84 pad 1: power_3v3-VCC -> power_3v3_digital
- C85 pad 1: power_3v3-VCC -> power_3v3_digital
- C94 pad 1: power_3v3-VCC -> power_3v3_digital
- C95 pad 1: power_3v3-VCC -> power_3v3_digital
- C96 pad 1: power_3v3-VCC -> power_3v3_digital
- C97 pad 1: power_3v3-VCC -> power_3v3_digital
- C98 pad 1: power_3v3-VCC -> power_3v3_digital
- C99 pad 1: power_3v3-VCC -> power_3v3_digital
- CN1 pad 12: gpio[26]-pins[23] -> logic_out-pins[23]
- CN1 pad 14: i2c_resistor_jumpers[2]-i2c_out-SCL -> smi_resistor_jumpers[1]-smi_out-SCL
- CN1 pad 18: reset_resistor_jumpers[0]-logic_out-SDA -> spi-SDA
- CN1 pad 23: i2cs[3]-SDA -> smi_resistor_jumpers[2]-smi_out-SDA
- CN1 pad 28: i2c_resistor_jumpers[1]-i2c_out-SCL -> smi_resistor_jumpers[0]-smi_out-SCL
- CN1 pad 29: reset_resistor_jumpers[2]-logic_out-SDA -> smi_resistor_jumpers[0]-smi_out-SDA
- CN1 pad 39: power_3v3-VCC -> power_3v3_digital
- CN1 pad 53: input-pins[94] -> power_led-pins[94]
- CN1 pad 57: power_5v-VCC -> power_5v
- CN1 pad 58: power_5v-VCC -> power_5v
- CN1 pad 59: power_5v-VCC -> power_5v
- CN1 pad 60: power_5v-VCC -> power_5v
- CN1 pad 61: power_5v-VCC -> power_5v
- CN1 pad 62: power_5v-VCC -> power_5v
- CN1 pad 77: i2cs[3]-SCL -> smi_resistor_jumpers[2]-smi_out-SCL
- CN1 pad 78: pins[44] -> nRESET
- CN1 pad 80: gpio[25]-pins[40] -> logic_out-pins[40]
- CN1 pad 83: logic_out-SCL -> spi-SCL
- CN1 pad 85: i2c_out-SDA -> smi_resistor_jumpers[1]-smi_out-SDA
- CN1 pad 90: activity_led_resistor-pins[20] -> activity_led-pins[20]
- CN2 pad 19: power_3v3-GND -> pins[37]_N
- D3 pad 5: power_5v-VCC -> power_5v
- F1 pad 2: power_5v-VCC -> power_5v
- J1000 pad 2: ADC1LN_P -> xlr_audio_input_connectors[0]-audio-audio_P
- J1000 pad 3: ADC1LP_N -> xlr_audio_input_connectors[0]-audio-audio_N
- J1001 pad 2: ADC1RN_P -> xlr_audio_input_connectors[1]-audio-audio_P
- J1001 pad 3: ADC1RP_N -> xlr_audio_input_connectors[1]-audio-audio_N
- Q1 pad 1: power_3v3-VCC -> power_3v3_digital
- R14 pad 1: power_3v3-VCC -> power_3v3_digital
- R15 pad 1: logic_out-SCL -> spi-SCL
- R15 pad 2: power_3v3-VCC -> power_3v3_digital
- R16 pad 1: reset_resistor_jumpers[0]-logic_out-SDA -> spi-SDA
- R16 pad 2: power_3v3-VCC -> power_3v3_digital
- R17 pad 1: i2c_resistor_jumpers[1]-i2c_out-SCL -> smi_resistor_jumpers[0]-smi_out-SCL
- R17 pad 2: power_3v3-VCC -> power_3v3_digital
- R18 pad 1: reset_resistor_jumpers[2]-logic_out-SDA -> smi_resistor_jumpers[0]-smi_out-SDA
- R18 pad 2: power_3v3-VCC -> power_3v3_digital
- R19 pad 1: i2c_resistor_jumpers[2]-i2c_out-SCL -> smi_resistor_jumpers[1]-smi_out-SCL
- R19 pad 2: power_3v3-VCC -> power_3v3_digital
- R2 pad 1: nPD_nRST -> RTS
- R20 pad 1: i2c_out-SDA -> smi_resistor_jumpers[1]-smi_out-SDA
- R20 pad 2: power_3v3-VCC -> power_3v3_digital
- R21 pad 1: switches[0]-i2c_mdio-SCL -> smi_resistor_jumpers[2]-smi_out-SCL
- R21 pad 2: logic_out-SCL -> power_3v3_digital
- R22 pad 1: switches[0]-i2c_mdio-SDA -> smi_resistor_jumpers[2]-smi_out-SDA
- R22 pad 2: reset_resistor_jumpers[0]-logic_out-SDA -> power_3v3_digital
- R23 pad 1: switches[1]-i2c_mdio-SCL -> switches[0]-i2c_mdio-SCL
- R23 pad 2: i2c_resistor_jumpers[1]-i2c_out-SCL -> smi_resistor_jumpers[0]-smi_out-SDA
- R24 pad 1: switches[1]-i2c_mdio-SDA -> switches[0]-i2c_mdio-SDA
- R24 pad 2: reset_resistor_jumpers[2]-logic_out-SDA -> smi_resistor_jumpers[0]-smi_out-SCL
- R25 pad 1: switches[2]-i2c_mdio-SCL -> switches[1]-i2c_mdio-SCL
- R25 pad 2: i2c_resistor_jumpers[2]-i2c_out-SCL -> smi_resistor_jumpers[1]-smi_out-SDA
- R26 pad 1: switches[2]-i2c_mdio-SDA -> switches[1]-i2c_mdio-SDA
- R26 pad 2: i2c_out-SDA -> smi_resistor_jumpers[1]-smi_out-SCL
- R27 pad 1: power_3v3-GND -> VDIV_OUTPUT
- R27 pad 2: regulator_24v_isolated_pos-power_out-GND -> power_3v3-GND
- R3 pad 1: activity_led-cathode -> power_3v3-GND
- R3 pad 2: activity_led_resistor-pins[20] -> power_out-GND
- R4 pad 1: cm5-cathode -> power_5v
- R4 pad 2: Y -> EN
- R44 pad 1: power_5v-VCC -> power_3v3_digital
- R44 pad 2: EN -> VDIV_OUTPUT
- R45 pad 1: VDIV_OUTPUT -> switches[2]-i2c_mdio-SCL
- R45 pad 2: power_3v3-GND -> smi_resistor_jumpers[2]-smi_out-SDA
- R46 pad 1: power_3v3-VCC -> switches[2]-i2c_mdio-SDA
- R46 pad 2: VDIV_OUTPUT -> smi_resistor_jumpers[2]-smi_out-SCL
- R47 pad 2: reset_resistor_jumpers[0]-logic_out-SDA -> logic_out-pins[40]
- R48 pad 2: logic_out-SCL -> logic_out-pins[23]
- R49 pad 2: reset_resistor_jumpers[2]-logic_out-SDA -> pins[47]
- R51 pad 2: power_3v3-VCC -> power_3v3_digital
- R53 pad 2: power_3v3-VCC -> power_3v3_digital
- R54 pad 2: power_3v3-VCC -> power_3v3_digital
- R56 pad 2: power_3v3-VCC -> power_3v3_digital
- R58 pad 2: power_3v3-VCC -> power_3v3_digital
- R59 pad 2: power_3v3-VCC -> power_3v3_digital
- R61 pad 2: power_3v3-VCC -> power_3v3_digital
- R63 pad 2: power_3v3-VCC -> power_3v3_digital
- R64 pad 2: power_3v3-VCC -> power_3v3_digital
- TP3 pad 1: power_3v3-VCC -> power_3v3_digital
- U1 pad 10: nPD_nRST -> RTS
- U10 pad 13: power_5v-VCC -> power_5v
- U10 pad 15: power_5v-VCC -> power_5v
- U10 pad 16: power_5v-VCC -> power_5v
- U11 pad 1: power_5v-VCC -> power_5v
- U11 pad 3: power_3v3-VCC -> power_3v3_digital
- U12 pad 1: regulator_24v_isolated_pos-power_out-GND -> power_out-GND
- U12 pad 20: regulator_24v_isolated_pos-power_out-GND -> power_out-GND
- U13 pad 10: regulator_24v_isolated_pos-power_out-GND -> power_out-GND
- U13 pad 11: regulator_24v_isolated_pos-power_out-GND -> power_out-GND
- U13 pad 4: regulator_24v_isolated_pos-power_out-GND -> power_out-GND
- U13 pad 5: regulator_24v_isolated_pos-power_out-GND -> power_out-GND
- U13 pad 6: regulator_24v_isolated_pos-power_out-GND -> power_out-GND
- U13 pad 7: regulator_24v_isolated_pos-power_out-GND -> power_out-GND
- U13 pad 9: regulator_24v_isolated_pos-power_out-GND -> power_out-GND
- U14 pad 1: power_5v-VCC -> power_5v
- U15 pad 1: power_5v-VCC -> power_5v
- U15 pad 4: regulator_24v_isolated_pos-power_out-GND -> power_out-GND
- U16 pad 3: power_5v-VCC -> power_5v
- U17 pad 18: power_3v3-VCC -> power_3v3_digital
- U17 pad 31: power_3v3-VCC -> power_3v3_digital
- U17 pad 37: power_3v3-VCC -> power_3v3_digital
- U17 pad 38: power_3v3-VCC -> power_3v3_digital
- U17 pad 48: power_3v3-VCC -> power_3v3_digital
- U17 pad 6: power_3v3-VCC -> power_3v3_digital
- U17 pad 8: power_3v3-VCC -> power_3v3_digital
- U18 pad 18: power_3v3-VCC -> power_3v3_digital
- U18 pad 31: power_3v3-VCC -> power_3v3_digital
- U18 pad 37: power_3v3-VCC -> power_3v3_digital
- U18 pad 38: power_3v3-VCC -> power_3v3_digital
- U18 pad 48: power_3v3-VCC -> power_3v3_digital
- U18 pad 6: power_3v3-VCC -> power_3v3_digital
- U18 pad 8: power_3v3-VCC -> power_3v3_digital
- U19 pad 18: power_3v3-VCC -> power_3v3_digital
- U19 pad 31: power_3v3-VCC -> power_3v3_digital
- U19 pad 37: power_3v3-VCC -> power_3v3_digital
- U19 pad 38: power_3v3-VCC -> power_3v3_digital
- U19 pad 48: power_3v3-VCC -> power_3v3_digital
- U19 pad 6: power_3v3-VCC -> power_3v3_digital
- U19 pad 8: power_3v3-VCC -> power_3v3_digital
- U20 pad 3: regulator_24v_isolated_pos-power_out-GND -> power_out-GND
- U21 pad 3: regulator_24v_isolated_pos-power_out-GND -> power_out-GND
- U22 pad 3: regulator_24v_isolated_pos-power_out-GND -> power_out-GND
- U23 pad 3: regulator_24v_isolated_pos-power_out-GND -> power_out-GND
- U24 pad 3: regulator_24v_isolated_pos-power_out-GND -> power_out-GND
- U25 pad 3: regulator_24v_isolated_pos-power_out-GND -> power_out-GND
- U26 pad 3: regulator_24v_isolated_pos-power_out-GND -> power_out-GND
- U27 pad 3: regulator_24v_isolated_pos-power_out-GND -> power_out-GND
- U3 pad : cm5-net-0 -> (no net)
- U4 pad : cm5-net-1 -> (no net)
- U5 pad : cm5-net-2 -> (no net)
- U6 pad : cm5-net-3 -> (no net)
- U7 pad 15: power_3v3-VCC -> power_3v3_digital
- U7 pad 18: power_3v3-VCC -> power_3v3_digital
- U7 pad 2: power_3v3-VCC -> power_3v3_digital
- U7 pad 24: reset_resistor_jumpers[0]-logic_out-SDA -> nRESET
- U7 pad 30: reset_resistor_jumpers[0]-logic_out-SDA -> spi-SDA
- U7 pad 31: logic_out-SCL -> spi-SCL
- U7 pad 38: power_3v3-VCC -> power_3v3_digital
- U7 pad 56: power_3v3-VCC -> power_3v3_digital
- U7 pad 7: power_3v3-VCC -> power_3v3_digital
- U8 pad 1: _1 -> spi-SCL
- U8 pad 10: _10 -> power_3v3-GND
- U8 pad 2: logic_out-SCL -> _2
- U8 pad 3: _3 -> spi-SDA
- U8 pad 4: reset_resistor_jumpers[0]-logic_out-SDA -> power-VCC
- U8 pad 5: reset_resistor_jumpers[0]-logic_out-SDA -> _5
- U8 pad 6: _6 -> nRESET
- U8 pad 9: power_3v3-GND -> _9
Routing:
- net regulator_24v_isolated_pos-power_out-GND: track 103.0 -> 0.00 mm, vias 8 -> 0
- net power_out-GND: track 0.00 -> 103.0 mm, vias 0 -> 8
- net power_3v3-VCC: track 82.9 -> 0.00 mm, vias 28 -> 0
- net power_3v3_digital: track 0.00 -> 79.4 mm, vias 0 -> 25
- net ADC1LP_N: track 0.00 -> 71.5 mm, vias 0 -> 1
- net ADC1LN_P: track 0.00 -> 69.6 mm, vias 0 -> 1
- net ADC1RP_N: track 0.00 -> 46.7 mm, vias 0 -> 1
- net ADC1RN_P: track 0.00 -> 44.7 mm, vias 0 -> 1
- net switches[2]-ethernets[4]-ETH_LED_SPEED: track 31.3 -> 0.00 mm, vias 1 -> 0
- net power_5v-VCC: track 29.8 -> 0.00 mm, vias 3 -> 0
- net switches[2]-ethernets[4]-ETH_LED_LINK: track 27.6 -> 0.00 mm, vias 1 -> 0
- net switches[2]-ethernets[4]-ETH_P0_N: track 21.4 -> 0.00 mm, vias 1 -> 0
- net switches[2]-ethernets[4]-ETH_P1_N: track 20.6 -> 0.00 mm, vias 1 -> 0
- net switches[2]-ethernets[4]-ETH_P3_P: track 20.3 -> 0.00 mm, vias 1 -> 0
- net switches[2]-ethernets[4]-ETH_P1_P: track 19.0 -> 0.00 mm, vias 1 -> 0
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- added copper zone on In1.Cu, net power_18v_pos
Other:
- copper layers 2 -> 4
- board text added: "HDI A"
- board text added: "HDI B"

Commit message: layout progress
Parts:
- moved C57 207.7 mm to (104.7, 150.1)
- moved C51 202.1 mm to (104.7, 153.3)
- moved C52 202.1 mm to (104.7, 151.5)
- moved C35 200.1 mm to (108.4, 130.6), turned to -90 degrees
- moved C36 198.1 mm to (110.2, 130.6), turned to -90 degrees
- moved R27 197.9 mm to (112.3, 133.0), turned to 180 degrees
- moved R44 195.9 mm to (114.2, 133.0), turned to 180 degrees
- moved U11 194.3 mm to (113.1, 129.9), turned to 0 degrees
- moved C54 194.0 mm to (104.8, 139.7)
- moved R4 193.1 mm to (112.6, 127.9), turned to 0 degrees
- moved C38 191.6 mm to (116.0, 130.5), turned to 90 degrees
- moved C56 191.4 mm to (104.8, 134.7)
- moved C37 189.7 mm to (117.8, 130.5), turned to 90 degrees
- moved C53 188.6 mm to (104.8, 136.1)
- moved C55 184.6 mm to (105.8, 128.8), turned to 90 degrees
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Routing:
- net ADC1LP_N: track 71.5 -> 7.12 mm
- net ADC1LN_P: track 69.6 -> 5.43 mm
- net ADC1RP_N: track 46.7 -> 3.57 mm
- net ADC1RN_P: track 44.7 -> 2.17 mm
Other:
- board size 359 x 111 mm -> 359 x 72.9 mm

Commit message: almost done with layout
Parts:
- added R67: 10Ω ±1% 62.5mW, UNI_ROYAL_0402WGF100JTCE:R0402, F.Cu at (0.00, 0.00)
- added R68: 10Ω ±1% 62.5mW, UNI_ROYAL_0402WGF100JTCE:R0402, F.Cu at (0.00, -10.0)
- added R69: 10Ω ±1% 62.5mW, UNI_ROYAL_0402WGF100JTCE:R0402, F.Cu at (0.00, -20.0)
- added R70: 10Ω ±1% 62.5mW, UNI_ROYAL_0402WGF100JTCE:R0402, F.Cu at (0.00, -30.0)
- added R71: 10Ω ±1% 62.5mW, UNI_ROYAL_0402WGF100JTCE:R0402, F.Cu at (0.00, -40.0)
- added R72: 10Ω ±1% 62.5mW, UNI_ROYAL_0402WGF100JTCE:R0402, F.Cu at (0.00, -50.0)
- moved R20 414.9 mm to (365.5, 146.5), turned to 90 degrees
- moved R19 411.2 mm to (365.5, 148.4), turned to -90 degrees
- moved R22 408.7 mm to (347.0, 146.0), turned to 90 degrees
- moved R21 404.5 mm to (347.0, 147.9), turned to -90 degrees
- moved R26 381.0 mm to (366.9, 147.6), turned to 180 degrees
- moved R25 376.6 mm to (366.9, 146.6), turned to 180 degrees
- moved R18 373.8 mm to (330.0, 145.5), turned to 90 degrees
- moved R17 370.0 mm to (330.0, 147.4), turned to -90 degrees
- moved R23 361.5 mm to (331.5, 145.9), turned to 180 degrees
- moved R46 355.2 mm to (348.5, 147.2), turned to 180 degrees
- moved R45 350.1 mm to (348.5, 146.2), turned to 180 degrees
- moved R24 349.2 mm to (331.5, 146.9), turned to 180 degrees
- moved R15 314.0 mm to (236.9, 148.3), turned to -90 degrees
- moved R16 281.1 mm to (239.5, 148.3), turned to -90 degrees
- moved R3 186.3 mm to (108.5, 149.0)
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Connections:
- net i2s_ins[0]-SCK renamed model-i2s_ins[0]-SCK-1
- net i2s_ins[0]-SD renamed model-i2s_ins[0]-SD-1
- net i2s_ins[0]-WS renamed model-i2s_ins[0]-WS-1
- net i2s_ins[1]-SD renamed model-i2s_ins[1]-SD-0
- C1 pad 2: power_3v3-GND -> GND
- C10 pad 2: power_3v3-GND -> GND
- C100 pad 2: power_3v3-GND -> GND
- C104 pad 1: power_out-GND -> GND
- C105 pad 2: power_out-GND -> GND
- C11 pad 2: power_3v3-GND -> GND
- C111 pad 1: power_out-GND -> GND
- C112 pad 2: power_out-GND -> GND
- C118 pad 1: power_out-GND -> GND
- C119 pad 2: power_out-GND -> GND
- C12 pad 2: power_3v3-GND -> GND
- C125 pad 1: power_out-GND -> GND
- C126 pad 2: power_out-GND -> GND
- C13 pad 2: power_3v3-GND -> GND
- C132 pad 1: power_out-GND -> GND
- C133 pad 2: power_out-GND -> GND
- C139 pad 1: power_out-GND -> GND
- C14 pad 2: power_3v3-GND -> GND
- C140 pad 2: power_out-GND -> GND
- C146 pad 1: power_out-GND -> GND
- C147 pad 2: power_out-GND -> GND
- C15 pad 2: power_3v3-GND -> GND
- C153 pad 1: power_out-GND -> GND
- C154 pad 2: power_out-GND -> GND
- C16 pad 2: power_3v3-GND -> GND
- C17 pad 2: power_3v3-GND -> GND
- C18 pad 2: power_3v3-GND -> GND
- C19 pad 2: power_3v3-GND -> GND
- C2 pad 2: power_3v3-GND -> GND
- C20 pad 2: power_3v3-GND -> GND
- C21 pad 2: power_3v3-GND -> GND
- C22 pad 2: power_3v3-GND -> GND
- C23 pad 2: power_3v3-GND -> GND
- C24 pad 2: power_3v3-GND -> GND
- C25 pad 2: power_3v3-GND -> GND
- C26 pad 2: power_3v3-GND -> GND
- C27 pad 2: power_3v3-GND -> GND
- C28 pad 2: power_3v3-GND -> GND
- C29 pad 2: power_3v3-GND -> GND
- C3 pad 2: power_3v3-GND -> GND
- C32 pad 2: power_3v3-GND -> GND
- C33 pad 2: power_3v3-GND -> GND
- C34 pad 2: power_3v3-GND -> GND
- C35 pad 2: power_3v3-GND -> GND
- C36 pad 2: power_3v3-GND -> GND
- C37 pad 2: power_3v3-GND -> GND
- C38 pad 2: power_3v3-GND -> GND
- C4 pad 2: power_3v3-GND -> GND
- C40 pad 1: power_out-GND -> GND
- C41 pad 1: power_out-GND -> GND
- C42 pad 2: power_out-GND -> GND
- C43 pad 2: power_out-GND -> GND
- C44 pad 2: power_out-GND -> GND
- C46 pad 2: power_out-GND -> GND
- C47 pad 2: power_3v3-GND -> GND
- C48 pad 2: power_3v3-GND -> GND
- C49 pad 2: power_3v3-GND -> GND
- C5 pad 2: power_3v3-GND -> GND
- C50 pad 2: power_3v3-GND -> GND
- C51 pad 2: power_3v3-GND -> GND
- C52 pad 2: power_3v3-GND -> GND
- C53 pad 2: power_3v3-GND -> GND
- C54 pad 2: power_3v3-GND -> GND
- C55 pad 2: power_3v3-GND -> GND
- C56 pad 2: power_3v3-GND -> GND
- C57 pad 2: power_3v3-GND -> GND
- C58 pad 2: power_3v3-GND -> GND
- C59 pad 2: power_3v3-GND -> GND
- C6 pad 2: power_3v3-GND -> GND
- C60 pad 2: power_3v3-GND -> GND
- C61 pad 2: power_3v3-GND -> GND
- C62 pad 2: power_3v3-GND -> GND
- C63 pad 2: power_3v3-GND -> GND
- C64 pad 2: power_3v3-GND -> GND
- C65 pad 2: power_3v3-GND -> GND
- C66 pad 2: power_3v3-GND -> GND
- C67 pad 2: power_3v3-GND -> GND
- C68 pad 2: power_3v3-GND -> GND
- C69 pad 2: power_3v3-GND -> GND
- C7 pad 2: power_3v3-GND -> GND
- C70 pad 2: power_3v3-GND -> GND
- C71 pad 2: power_3v3-GND -> GND
- C72 pad 2: power_3v3-GND -> GND
- C73 pad 2: power_3v3-GND -> GND
- C74 pad 2: power_3v3-GND -> GND
- C75 pad 2: power_3v3-GND -> GND
- C76 pad 2: power_3v3-GND -> GND
- C77 pad 2: power_3v3-GND -> GND
- C78 pad 2: power_3v3-GND -> GND
- C79 pad 2: power_3v3-GND -> GND
- C8 pad 2: power_3v3-GND -> GND
- C80 pad 2: power_3v3-GND -> GND
- C81 pad 2: power_3v3-GND -> GND
- C82 pad 2: power_3v3-GND -> GND
- C83 pad 2: power_3v3-GND -> GND
- C84 pad 2: power_3v3-GND -> GND
- C85 pad 2: power_3v3-GND -> GND
- C86 pad 2: power_3v3-GND -> GND
- C87 pad 2: power_3v3-GND -> GND
- C88 pad 2: power_3v3-GND -> GND
- C89 pad 2: power_3v3-GND -> GND
- C9 pad 2: power_3v3-GND -> GND
- C90 pad 2: power_3v3-GND -> GND
- C91 pad 2: power_3v3-GND -> GND
- C92 pad 2: power_3v3-GND -> GND
- C93 pad 2: power_3v3-GND -> GND
- C94 pad 2: power_3v3-GND -> GND
- C95 pad 2: power_3v3-GND -> GND
- C96 pad 2: power_3v3-GND -> GND
- C97 pad 2: power_3v3-GND -> GND
- C98 pad 2: power_3v3-GND -> GND
- C99 pad 2: power_3v3-GND -> GND
- CN1 pad 1: power_3v3-GND -> GND
- CN1 pad 100: power_3v3-GND -> GND
- CN1 pad 11: power_3v3-GND -> GND
- CN1 pad 16: power_3v3-GND -> GND
- CN1 pad 21: power_3v3-GND -> GND
- CN1 pad 26: power_3v3-GND -> GND
- CN1 pad 30: power_3v3-GND -> GND
- CN1 pad 33: power_3v3-GND -> GND
- CN1 pad 37: power_3v3-GND -> GND
- CN1 pad 4: power_3v3-GND -> GND
- CN1 pad 49: power_3v3-GND -> GND
- CN1 pad 65: power_3v3-GND -> GND
- CN1 pad 68: power_3v3-GND -> GND
- CN1 pad 7: power_3v3-GND -> GND
- CN1 pad 71: power_3v3-GND -> GND
- CN1 pad 74: power_3v3-GND -> GND
- CN1 pad 79: power_3v3-GND -> GND
- CN1 pad 84: power_3v3-GND -> GND
- CN1 pad 89: power_3v3-GND -> GND
- CN1 pad 94: power_3v3-GND -> GND
- CN1 pad 97: power_3v3-GND -> GND
- CN2 pad 10: power_3v3-GND -> GND
- CN2 pad 13: power_3v3-GND -> GND
- CN2 pad 16: power_3v3-GND -> GND
- CN2 pad 22: power_3v3-GND -> GND
- CN2 pad 28: power_3v3-GND -> GND
- CN2 pad 31: power_3v3-GND -> GND
- CN2 pad 34: power_3v3-GND -> GND
- CN2 pad 37: power_3v3-GND -> GND
- CN2 pad 4: power_3v3-GND -> GND
- CN2 pad 40: power_3v3-GND -> GND
- CN2 pad 43: power_3v3-GND -> GND
- CN2 pad 46: power_3v3-GND -> GND
- CN2 pad 49: power_3v3-GND -> GND
- CN2 pad 52: power_3v3-GND -> GND
- CN2 pad 55: power_3v3-GND -> GND
- CN2 pad 58: power_3v3-GND -> GND
- CN2 pad 61: power_3v3-GND -> GND
- CN2 pad 64: power_3v3-GND -> GND
- CN2 pad 67: power_3v3-GND -> GND
- CN2 pad 7: power_3v3-GND -> GND
- CN2 pad 70: power_3v3-GND -> GND
- CN2 pad 73: power_3v3-GND -> GND
- CN2 pad 82: power_3v3-GND -> GND
- CN2 pad 85: power_3v3-GND -> GND
- CN2 pad 88: power_3v3-GND -> GND
- CN2 pad 91: power_3v3-GND -> GND
- CN2 pad 94: power_3v3-GND -> GND
- CN2 pad 97: power_3v3-GND -> GND
- D3 pad 2: power_3v3-GND -> GND
- J1000 pad : footprint-net-13 -> footprint-net-15
- J1001 pad : footprint-net-14 -> footprint-net-16
- J1002 pad : footprint-net-15 -> footprint-net-17
- J1003 pad : footprint-net-16 -> footprint-net-18
- J1004 pad : footprint-net-17 -> footprint-net-19
- J1005 pad : footprint-net-18 -> footprint-net-20
- J1006 pad : footprint-net-19 -> footprint-net-21
- J1007 pad : footprint-net-20 -> footprint-net-22
- J1008 pad : footprint-net-21 -> footprint-net-23
- J1009 pad : footprint-net-22 -> footprint-net-24
- J1010 pad : footprint-net-23 -> footprint-net-25
- J1011 pad : footprint-net-24 -> footprint-net-26
- R2 pad 2: power_3v3-GND -> GND
- R27 pad 2: power_3v3-GND -> GND
- R3 pad 1: power_3v3-GND -> footprint-net-1
- R3 pad 2: power_out-GND -> footprint-net-2
- R50 pad 2: power_3v3-GND -> GND
- R52 pad 2: power_3v3-GND -> GND
- R55 pad 2: power_3v3-GND -> GND
- R57 pad 2: power_3v3-GND -> GND
- R60 pad 2: power_3v3-GND -> GND
- R62 pad 2: power_3v3-GND -> GND
- R65 pad 2: power_3v3-GND -> GND
- R66 pad 2: power_3v3-GND -> GND
- TP2 pad 1: power_3v3-GND -> GND
- U1 pad 1: power_3v3-GND -> GND
- U1 pad 12: power_3v3-GND -> GND
- U1 pad 16: model-i2s_outs[1]-SD-0 -> model-i2s_ins[0]-SD-0
- U1 pad 17: i2s_outs[1]-SCK -> model-i2s_ins[0]-SCK-0
- U1 pad 18: i2s_outs[1]-WS -> model-i2s_ins[0]-WS-0
- U1 pad 19: model-i2s_outs[1]-SD-1 -> model-i2s_outs[1]-SD-0
- U1 pad 25: power_3v3-GND -> GND
- U1 pad 32: power_3v3-GND -> GND
- U1 pad 34: power_3v3-GND -> GND
- U1 pad 36: power_3v3-GND -> GND
- U1 pad 4: power_3v3-GND -> GND
- U10 pad 11: power_3v3-GND -> GND
- U10 pad 12: power_3v3-GND -> GND
- U10 pad 17: footprint-net-11 -> footprint-net-13
- U10 pad 18: footprint-net-12 -> footprint-net-14
- U10 pad 19: footprint-net-9 -> footprint-net-11
- U10 pad 2: footprint-net-10 -> footprint-net-12
- U10 pad 21: footprint-EP-2 -> GND
- U10 pad 7: power_3v3-GND -> GND
- U10 pad 8: power_3v3-GND -> GND
- U11 pad 4: power_3v3-GND -> GND
- U12 pad 1: power_out-GND -> GND
- U12 pad 17: footprint-net-3 -> footprint-net-5
- U12 pad 18: footprint-net-4 -> footprint-net-6
- U12 pad 19: footprint-net-1 -> footprint-net-3
- U12 pad 2: footprint-net-2 -> footprint-net-4
- U12 pad 20: power_out-GND -> GND
- U12 pad 21: footprint-EP-0 -> power_18v_neg
- U13 pad 10: power_out-GND -> GND
- U13 pad 11: power_out-GND -> GND
- U13 pad 17: footprint-net-7 -> footprint-net-9
- U13 pad 18: footprint-net-8 -> footprint-net-10
- U13 pad 19: footprint-net-5 -> footprint-net-7
- U13 pad 2: footprint-net-6 -> footprint-net-8
- U13 pad 21: footprint-EP-1 -> GND
- U13 pad 4: power_out-GND -> GND
- U13 pad 5: power_out-GND -> GND
- U13 pad 6: power_out-GND -> GND
- U13 pad 7: power_out-GND -> GND
- U13 pad 9: power_out-GND -> GND
- U14 pad 2: power_3v3-GND -> GND
- U15 pad 2: power_3v3-GND -> GND
- U15 pad 4: power_out-GND -> GND
- U16 pad 4: power_3v3-GND -> GND
- U17 pad 49: power_3v3-GND -> GND
- U18 pad 49: power_3v3-GND -> GND
- U19 pad 49: power_3v3-GND -> GND
- U20 pad 3: power_out-GND -> GND
- U21 pad 3: power_out-GND -> GND
- U22 pad 3: power_out-GND -> GND
- U23 pad 3: power_out-GND -> GND
- U24 pad 3: power_out-GND -> GND
- U25 pad 3: power_out-GND -> GND
- U26 pad 3: power_out-GND -> GND
- U27 pad 3: power_out-GND -> GND
- U3 pad 1: power_3v3-GND -> GND
- U3 pad 2: power_3v3-GND -> GND
- U3 pad 3: power_3v3-GND -> GND
- U3 pad 4: power_3v3-GND -> GND
- U4 pad 1: power_3v3-GND -> GND
- U4 pad 2: power_3v3-GND -> GND
- U4 pad 3: power_3v3-GND -> GND
- U4 pad 4: power_3v3-GND -> GND
- U5 pad 1: power_3v3-GND -> GND
- U5 pad 2: power_3v3-GND -> GND
- U5 pad 3: power_3v3-GND -> GND
- U5 pad 4: power_3v3-GND -> GND
- U6 pad 1: power_3v3-GND -> GND
- U6 pad 2: power_3v3-GND -> GND
- U6 pad 3: power_3v3-GND -> GND
- U6 pad 4: power_3v3-GND -> GND
- U7 pad 1: power_3v3-GND -> GND
- U7 pad 14: power_3v3-GND -> GND
- U7 pad 17: power_3v3-GND -> GND
- U7 pad 19: power_3v3-GND -> GND
- U7 pad 25: power_3v3-GND -> GND
- U7 pad 36: power_3v3-GND -> GND
- U7 pad 37: power_3v3-GND -> GND
- U7 pad 44: model-i2s_outs[1]-SD-0 -> model-i2s_outs[1]-SD-1
- U7 pad 54: power_3v3-GND -> GND
- U7 pad 55: power_3v3-GND -> GND
- U7 pad 6: power_3v3-GND -> GND
- U7 pad 60: model-i2s_outs[0]-SCK-0 -> i2s_ins[1]-SCK
- U7 pad 61: model-i2s_outs[0]-WS-0 -> i2s_ins[1]-WS
- U7 pad 62: model-i2s_outs[0]-SD-0 -> model-i2s_ins[1]-SD-1
- U7 pad 72: power_3v3-GND -> GND
- U7 pad 73: power_3v3-GND -> GND
- U8 pad 10: power_3v3-GND -> GND
- U9 pad 100: power_3v3-GND -> GND
- U9 pad 101: power_3v3-GND -> GND
- U9 pad 102: power_3v3-GND -> GND
- U9 pad 11: power_3v3-GND -> GND
- U9 pad 21: power_3v3-GND -> GND
- U9 pad 23: power_3v3-GND -> GND
- U9 pad 33: power_3v3-GND -> GND
- U9 pad 35: power_3v3-GND -> GND
- U9 pad 45: power_3v3-GND -> GND
- U9 pad 47: power_3v3-GND -> GND
- U9 pad 58: power_3v3-GND -> GND
- U9 pad 60: power_3v3-GND -> GND
- U9 pad 70: power_3v3-GND -> GND
- U9 pad 72: power_3v3-GND -> GND
- U9 pad 82: power_3v3-GND -> GND
- U9 pad 84: power_3v3-GND -> GND
- U9 pad 9: power_3v3-GND -> GND
- U9 pad 94: power_3v3-GND -> GND
- U9 pad 96: power_3v3-GND -> GND
- U9 pad 97: power_3v3-GND -> GND
- U9 pad 98: power_3v3-GND -> GND
- U9 pad 99: power_3v3-GND -> GND
- USB1 pad : (no net) -> connector-net
- USB1 pad 1: power_3v3-GND -> GND
- USB1 pad 12: power_3v3-GND -> GND
- USB1 pad 13: power_3v3-GND -> GND
- USB1 pad 14: power_3v3-GND -> GND
- USB1 pad 15: power_3v3-GND -> GND
- USB1 pad 16: power_3v3-GND -> GND
- X1 pad 2: power_3v3-GND -> GND
- X1 pad 4: power_3v3-GND -> GND
- X2 pad 2: power_3v3-GND -> GND
- X2 pad 4: power_3v3-GND -> GND
- X3 pad 2: power_3v3-GND -> GND
- X3 pad 4: power_3v3-GND -> GND
- X4 pad 2: power_3v3-GND -> GND
- X4 pad 4: power_3v3-GND -> GND
Routing:
- net GND: track 0.00 -> 314.3 mm, vias 0 -> 91
- net power_3v3-GND: track 174.1 -> 0.00 mm, vias 83 -> 0
- net xlr_audio_input_connectors[0]-audio-audio_N: track 0.00 -> 109.3 mm
- net power_out-GND: track 103.0 -> 0.00 mm, vias 8 -> 0
- net OL1: track 0.00 -> 101.9 mm, vias 0 -> 2
- net ADC1LP_N: track 7.12 -> 105.5 mm
- net ADC1RN_P: track 2.17 -> 98.5 mm
- net xlr_audio_input_connectors[0]-audio-audio_P: track 0.00 -> 94.5 mm
- net ADC1RP_N: track 3.57 -> 96.3 mm
- net OR1: track 0.00 -> 92.3 mm, vias 0 -> 2
- net ADC1LN_P: track 5.43 -> 95.8 mm
- net OL2: track 0.00 -> 82.6 mm, vias 0 -> 2
- net OR2: track 0.00 -> 73.0 mm, vias 0 -> 2
- net xlr_audio_output_connectors[0]-audio-audio_P: track 10.6 -> 79.0 mm
- net xlr_audio_input_connectors[1]-audio-audio_N: track 0.00 -> 67.0 mm
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- added copper zone on B.Cu, net footprint-net-1
- added copper zone on F.Cu, net footprint-net-1
- added copper zone on In2.Cu, net footprint-net-1
- added copper zone on In1.Cu, net power_18v_neg
- added copper zone on F.Cu, net power_5v
- removed copper zone on B.Cu, net power_3v3-GND
- removed copper zone on F.Cu, net power_3v3-GND
Other:
- board text added: "SMI_SW_0"
- board text added: "SMI_SW_1"
- board text added: "SMI_SW_2"
