File: projects/dsp/layouts/default/default.kicad_pcb (KiCad board)
At the start: 4 copper layers, 359 x 73.8 mm, 412 parts

Commit message: shipped board
Connections:
- J1000 pad : (no net) -> footprint-net-15
- J1001 pad : (no net) -> footprint-net-16
- J1002 pad : (no net) -> footprint-net-17
- J1003 pad : (no net) -> footprint-net-18
- J1004 pad : (no net) -> footprint-net-19
- J1005 pad : (no net) -> footprint-net-20
- J1006 pad : (no net) -> footprint-net-21
- J1007 pad : (no net) -> footprint-net-22
- J1010 pad : (no net) -> footprint-net-23
- J1011 pad : (no net) -> footprint-net-24
- PS1 pad : (no net) -> ethercon_output_connectors[0]-net
- PS2 pad : (no net) -> ethercon_output_connectors[1]-net
- U3 pad 3: GND -> (no net)
- U3 pad 4: GND -> (no net)
- U4 pad 3: GND -> (no net)
- U4 pad 4: GND -> (no net)
- U5 pad 3: GND -> (no net)
- U5 pad 4: GND -> (no net)
- U6 pad 3: GND -> (no net)
- U6 pad 4: GND -> (no net)
- U9 pad : (no net) -> footprint-net-0
- USB1 pad : (no net) -> connector-net
Routing:
- net footprint-net-0: track 57.1 -> 0.00 mm
- net 593: track 0.00 -> 57.1 mm
- net footprint-net-24: track 14.1 -> 0.00 mm
- net 589: track 0.00 -> 14.1 mm
- net footprint-net-15: track 14.1 -> 0.00 mm
- net 583: track 0.00 -> 14.1 mm
- net footprint-net-16: track 14.1 -> 0.00 mm
- net 592: track 0.00 -> 14.1 mm
- net ethercon_output_connectors[0]-net: track 13.8 -> 0.00 mm
- net 588: track 0.00 -> 13.8 mm
- net ethercon_output_connectors[1]-net: track 13.8 -> 0.00 mm
- net 591: track 0.00 -> 13.8 mm
- net footprint-net-23: track 9.72 -> 0.00 mm
- net footprint-net-20: track 9.72 -> 0.00 mm
- net 585: track 0.00 -> 9.72 mm
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